File: Boards/Netzteil/12V_Supply/12V_Supply.kicad_pcb (KiCad board)
At the start: 2 copper layers, 100 x 80 mm, 24 parts, among them P1 230V_AC, P2 12V_DC_1, P3 12V_DC_2, P4 Relais, P5 12V_DC_3, P6 12V_DC_4, P7 Relais, U1 LM555N, U2 LM7812CT

Commit message: Updated Layout
Parts:
- moved C5 3.68 mm to (167.6, 98.4), turned to 270 degrees
- moved R2 2.01 mm to (153.0, 101.0), turned to 180 degrees
Routing:
- net Net-(C1-Pad1): track 60.0 -> 47.4 mm
- net Net-(D1-Pad1): track 3.43 -> 7.93 mm
- net +12V: track 205.5 -> 203.0 mm
- net Net-(D4-Pad1): track 15.6 -> 13.8 mm

Commit message: Work in Progress
Parts:
- moved C5 0.79 mm to (168.4, 98.4)
Routing:
- net Net-(F1-Pad1): track 50.2 -> 44.4 mm
- net Net-(D1-Pad3): track 20.5 -> 19.9 mm
Changed lines of the file:
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@@
-(kicad_pcb (version 4) (host pcbnew 4.0.2-stable)
+(kicad_pcb (version 4) (host pcbnew 4.0.3-stable)
   (general
     (links 40)
     (no_connects 0)
-    (area 92.514 54.247 193.354301 150.327)
+    (area 92.514 54.397 193.354301 150.427)
     (thickness 1.6)
     (drawings 0)
-    (tracks 88)
+    (tracks 86)
     (zones 0)
     (modules 24)
@@
   )
   (module w_capacitors:CP_8x15mm (layer F.Cu)
-    (at 167.64 98.425 270)
+    (at 168.43 98.425 270)
     (descr "Capacitor, pol, cyl 8x15mm")
     (fp_text reference C5 (at 0 -5.6 270) (layer F.SilkS)
@@
     )
   )
-  (segment (start 158.115 100.965) (end 158.115 100.736141) (width 1) (layer B.Cu) (net 1))
-  (segment (start 158.115 100.736141) (end 158.496 100.355141) (width 1) (layer B.Cu) (net 1))
-  (segment (start 158.496 100.355141) (end 158.496 83.312) (width 1) (layer B.Cu) (net 1))
+  (segment (start 158.115 100.965) (end 158.109934 100.959934) (width 1) (layer B.Cu) (net 1))
+  (segment (start 158.109934 100.959934) (end 158.109934 83.698066) (width 1) (layer B.Cu) (net 1))
+  (segment (start 158.109934 83.698066) (end 158.496 83.312) (width 1) (layer B.Cu) (net 1))
   (segment (start 158.055 114.935) (end 158.055 101.025) (width 1) (layer B.Cu) (net 1))
   (segment (start 158.055 101.025) (end 158.115 100.965) (width 1) (layer B.Cu) (net 1))
@@
   (segment (start 178.7779 117.35816) (end 178.9049 117.48516) (width 1) (layer B.Cu) (net 2) (status 30))
   (segment (start 178.9049 105.03916) (end 178.7779 105.16616) (width 1) (layer B.Cu) (net 2) (status 30))
-  (segment (start 165.89 98.425) (end 165.89 96.414747) (width 1) (layer B.Cu) (net 3))
-  (segment (start 165.89 96.414747) (end 166.624 95.680747) (width 1) (layer B.Cu) (net 3))
+  (segment (start 163.27 132.08) (end 163.27 125.939046) (width 1) (layer B.Cu) (net 3))
+  (segment (start 163.27 125.939046) (end 166.624 122.585046) (width 1) (layer B.Cu) (net 3))
+  (segment (start 166.624 122.585046) (end 166.624 95.680747) (width 1) (layer B.Cu) (net 3))
   (segment (start 166.624 95.680747) (end 166.624 83.312) (width 1) (layer B.Cu) (net 3))
-  (segment (start 163.27 132.08) (end 163.27 125.939046) (width 1) (layer B.Cu) (net 3))
-  (segment (start 163.27 125.939046) (end 165.89 123.319046) (width 1) (layer B.Cu) (net 3))
-  (segment (start 165.89 123.319046) (end 165.89 100.928254) (width 1) (layer B.Cu) (net 3))
-  (segment (start 165.89 100.928254) (end 165.89 98.425) (width 1) (layer B.Cu) (net 3))
   (segment (start 113.03 127.254) (end 113.071011 127.212989) (width 1) (layer B.Cu) (net 3))
   (segment (start 113.071011 127.212989) (end 113.071011 124.727535) (width 1) (layer B.Cu) (net 3))
@@
   (segment (start 128.524 121.654) (end 128.282 121.412) (width 0.5) (layer B.Cu) (net 4) (status 30))
   (segment (start 127.774 121.92) (end 128.282 121.412) (width 0.5) (layer B.Cu) (net 4) (status 30))
-  (segment (start 142.621 88.9) (end 139.7 88.9) (width 1) (layer B.Cu) (net 5) (status 10))
-  (segment (start 135.3439 84.5439) (end 135.3439 73.152) (width 1) (layer B.Cu) (net 5) (status 20))
-  (segment (start 139.7 88.9) (end 135.3439 84.5439) (width 1) (layer B.Cu) (net 5))
+  (segment (start 142.621 88.9) (end 140.648572 88.9) (width 1) (layer B.Cu) (net 5))
+  (segment (start 140.648572 88.9) (end 135.3439 83.595328) (width 1) (layer B.Cu) (net 5))
+  (segment (start 135.3439 83.595328) (end 135.3439 73.152) (width 1) (layer B.Cu) (net 5))
   (segment (start 118.11 134.874) (end 118.11 136.858029) (width 1) (layer B.Cu) (net 6))
   (segment (start 118.11 136.858029) (end 118.930888 137.678917) (width 1) (layer B.Cu) (net 6))
@@
   (segment (start 134.874 94.234) (end 142.367 94.234) (width 1) (layer B.Cu) (net 8) (status 30))
   (segment (start 142.367 94.234) (end 142.621 93.98) (width 1) (layer B.Cu) (net 8) (status 30))
-  (segment (start 134.874 104.394) (end 131.826 104.394) (width 1) (layer B.Cu) (net 9) (status 10))
-  (segment (start 127 73.152) (end 113.5761 73.152) (width 1) (layer B.Cu) (net 9) (status 20))
-  (segment (start 129.032 75.184) (end 127 73.152) (width 1) (layer B.Cu) (net 9))
-  (segment (start 129.032 101.6) (end 129.032 75.184) (width 1) (layer B.Cu) (net 9))
-  (segment (start 131.826 104.394) (end 129.032 101.6) (width 1) (layer B.Cu) (net 9))
+  (segment (start 134.874 104.394) (end 132.970782 104.394) (width 1) (layer B.Cu) (net 9))
+  (segment (start 132.970782 104.394) (end 126.348545 97.771763) (width 1) (layer B.Cu) (net 9))
+  (segment (start 126.348545 97.771763) (end 126.348545 81.290153) (width 1) (layer B.Cu) (net 9))
+  (segment (start 126.348545 81.290153) (end 118.210392 73.152) (width 1) (layer B.Cu) (net 9))
+  (segment (start 118.210392 73.152) (end 113.5761 73.152) (width 1) (layer B.Cu) (net 9))
   (segment (start 134.874 104.394) (end 134.366 104.394) (width 1) (layer B.Cu) (net 9) (status 30))
   (segment (start 102.108 103.886) (end 110.236 103.886) (width 1) (layer B.Cu) (net 10) (status 10))
@@
   (segment (start 102.108 96.266) (end 108.712 96.266) (width 1) (layer B.Cu) (net 11) (status 10))
   (segment (start 108.712 96.266) (end 115.824 89.154) (width 1) (layer B.Cu) (net 11) (status 20))
-  (segment (start 150.241 93.98) (end 150.241 98.679) (width 1) (layer B.Cu) (net 12))
-  (segment (start 150.241 98.679) (end 147.955 100.965) (width 1) (layer B.Cu) (net 12))
+  (segment (start 150.241 93.98) (end 150.241 96.295067) (width 1) (layer B.Cu) (net 12))
+  (segment (start 150.241 96.295067) (end 147.955 98.581067) (width 1) (layer B.Cu) (net 12))
+  (segment (start 147.955 98.581067) (end 147.955 100.965) (width 1) (layer B.Cu) (net 12))
   (zone (net 2) (net_name GND) (layer B.Cu) (hatch edge 0.508)
     (connect_pads (clearance 0.5))
@@
     (polygon
       (pts
-        (xy 192.024 141.224) (xy 93.472 141.224) (xy 93.472 62.484) (xy 192.024 62.484) (xy 192.024 141.224)
+        (xy 192.024 141.224) (xy 93.472 141.224) (xy 93.472 62.484) (xy 192.024 62.484)
       )
     )
@@
     (polygon
       (pts
-        (xy 121.92 114.3) (xy 92.964 114.3) (xy 92.964 84.836) (xy 121.92 84.836) (xy 121.92 114.3)
+        (xy 123.952 115.824) (xy 92.964 115.824) (xy 92.964 82.804) (xy 123.952 82.804) (xy 123.952 114.3)
       )
     )

Commit message: Work in Progress
Parts:
- added D5: LED, LEDs:LED_D3.0mm, F.Cu at (169.5, 135.9)
- added R3: 47k, Resistors_THT:R_Axial_DIN0207_L6.3mm_D2.5mm_P10.16mm_Horizontal, F.Cu at (161.9, 123.2)
- C4: value 1µF -> 200µF
- R1: value 18k -> 47k
- moved R2 4.44 mm to (148.6, 101.0)
Routing:
- net Net-(C1-Pad1): track 47.4 -> 64.9 mm
- net Net-(D5-Pad2): track 0.00 -> 14.5 mm
- net Net-(D4-Pad2): track 31.7 -> 44.3 mm
- net +12V: track 203.0 -> 199.1 mm
- net Net-(D1-Pad1): track 7.93 -> 11.5 mm
- net Net-(F1-Pad1): track 44.4 -> 47.9 mm
