File: Boards/Netzteil/12V_Supply/12V_Supply.sch (KiCad schematic (older format))
At the start: 22 parts, among them P1 230V_AC, P2 12V_DC_1, P3 12V_DC_2, P4 Relais, P5 12V_DC_3, P6 12V_DC_4, P7 Relais, U1 LM555N, U2 LM7812CT

Commit message: Work in Progress
Parts:
- U1: symbol LM555N -> LM555N-RESCUE-12V_Supply
Changed lines of the file:
@@
 EESchema Schematic File Version 2
+LIBS:12V_Supply-rescue
 LIBS:power
 LIBS:device
@@
 Connection ~ 7150 2200
 $Comp
-L GND #PWR9
+L GND-RESCUE-12V_Supply #PWR9
 U 1 1 55C54F23
 P 7450 3150
@@
 $EndComp
 $Comp
-L GND #PWR2
+L GND-RESCUE-12V_Supply #PWR2
 U 1 1 55C54FA5
 P 7450 2500
@@
 $EndComp
 $Comp
-L GND #PWR8
+L GND-RESCUE-12V_Supply #PWR8
 U 1 1 55C54FCF
 P 6550 2600
@@
 $EndComp
 $Comp
-L GND #PWR7
+L GND-RESCUE-12V_Supply #PWR7
 U 1 1 55C55002
 P 5750 2600
@@
 $EndComp
 $Comp
-L GND #PWR6
+L GND-RESCUE-12V_Supply #PWR6
 U 1 1 55C5507B
 P 5100 2600
@@
 $EndComp
 $Comp
-L GND #PWR5
+L GND-RESCUE-12V_Supply #PWR5
 U 1 1 55C550A7
 P 4350 2600
@@
 $EndComp
 $Comp
-L GND #PWR4
+L GND-RESCUE-12V_Supply #PWR4
 U 1 1 55C550D3
 P 3650 2600
@@
 $EndComp
 $Comp
-L GND #PWR3
+L GND-RESCUE-12V_Supply #PWR3
 U 1 1 55C550FF
 P 2300 2600
@@
 $EndComp
 $Comp
-L LM555N U1
+L LM555N-RESCUE-12V_Supply U1
 U 1 1 55C55C2A
 P 5050 4850
@@
 $EndComp
 $Comp
-L GND #PWR13
+L GND-RESCUE-12V_Supply #PWR13
 U 1 1 55C5698D
 P 5050 5400
@@
 Connection ~ 5950 4300
 $Comp
-L GND #PWR14
+L GND-RESCUE-12V_Supply #PWR14
 U 1 1 55C57D8C
 P 5950 5450
@@
 	7150 3300 7450 3300
 $Comp
-L GND #PWR10
+L GND-RESCUE-12V_Supply #PWR10
 U 1 1 55C680B0
 P 7450 3650
@@
 	7150 3850 7450 3850
 $Comp
-L GND #PWR12
+L GND-RESCUE-12V_Supply #PWR12
 U 1 1 55C68115
 P 7450 4200

Commit message: Work in Progress
Parts:
- added D5: LED, LEDs:LED_D3.0mm, symbol LED
- added R3: 47k, Resistors_THT:R_Axial_DIN0207_L6.3mm_D2.5mm_P10.16mm_Horizontal, symbol R
- C2, C3: footprint Capacitors_ThroughHole:C_Disc_D3_P2.5 -> Capacitors_THT:C_Disc_D3.0mm_W2.0mm_P2.50mm
- C4: value 1µF -> 200µF
- P2, P3, P5, P6: footprint MiniUniversalMate-N-LokSockets_13Aug2012:MiniUniversalMate-N-LokSocket_2PinVertical_12Aug2012 -> Connectors_Mini-Universal:MiniUniversalMate-N-LokSocket_2PinVertical
- R1: value 18k -> 47k; footprint Resistors_ThroughHole:Resistor_Horizontal_RM10mm -> Resistors_THT:R_Axial_DIN0207_L6.3mm_D2.5mm_P10.16mm_Horizontal
- R2: footprint Resistors_ThroughHole:Resistor_Horizontal_RM10mm -> Resistors_THT:R_Axial_DIN0207_L6.3mm_D2.5mm_P10.16mm_Horizontal
Connections:
- net +12V: now also R3.1
- net at D4.2 (A), P4.2 (P2), P7.2 (P2): now also D5.1 (K)
- new net: D5.2 (A), R3.2
Other:
- note added: "Power-On-Delay\nca. 10s\n(Tdelay = 1.1 * C * R)"
- note removed: "Power-On-Delay\n20s\n(Tdelay = 1.1 * C * R)"
- moved on the sheet: D4
Changed lines of the file:
@@
 LIBS:ftdi
 LIBS:gennum
-LIBS:graphic
 LIBS:hc11
 LIBS:ir
 LIBS:Lattice
-LIBS:logo
 LIBS:maxim
 LIBS:microchip_dspic33dsc
@@
 F 0 "C2" H 4375 2450 50  0000 L CNN
 F 1 "100nF / 63V" H 4375 2250 50  0000 L CNN
-F 2 "Capacitors_ThroughHole:C_Disc_D3_P2.5" H 4388 2200 30  0001 C CNN
+F 2 "Capacitors_THT:C_Disc_D3.0mm_W2.0mm_P2.50mm" H 4388 2200 30  0001 C CNN
 F 3 "" H 4350 2350 60  0000 C CNN
 	1    4350 2350
@@
 F 0 "C3" H 5775 2450 50  0000 L CNN
 F 1 "100nF / 16V" H 5775 2250 50  0000 L CNN
-F 2 "Capacitors_ThroughHole:C_Disc_D3_P2.5" H 5788 2200 30  0001 C CNN
+F 2 "Capacitors_THT:C_Disc_D3.0mm_W2.0mm_P2.50mm" H 5788 2200 30  0001 C CNN
 F 3 "" H 5750 2350 60  0000 C CNN
 	1    5750 2350
@@
 F 0 "P2" V 7750 2300 40  0000 C CNN
 F 1 "12V_DC_1" V 7850 2300 40  0000 C CNN
-F 2 "MiniUniversalMate-N-LokSockets_13Aug2012:MiniUniversalMate-N-LokSocket_2PinVertical_12Aug2012" H 7800 2300 60  0001 C CNN
+F 2 "Connectors_Mini-Universal:MiniUniversalMate-N-LokSocket_2PinVertical" H 7800 2300 60  0001 C CNN
 F 3 "" H 7800 2300 60  0000 C CNN
 	1    7800 2300
@@
 F 0 "P3" V 7750 2900 40  0000 C CNN
 F 1 "12V_DC_2" V 7850 2900 40  0000 C CNN
-F 2 "MiniUniversalMate-N-LokSockets_13Aug2012:MiniUniversalMate-N-LokSocket_2PinVertical_12Aug2012" H 7800 2900 60  0001 C CNN
+F 2 "Connectors_Mini-Universal:MiniUniversalMate-N-LokSocket_2PinVertical" H 7800 2900 60  0001 C CNN
 F 3 "" H 7800 2900 60  0000 C CNN
 	1    7800 2900
@@
 Connection ~ 7150 2200
 $Comp
-L GND-RESCUE-12V_Supply #PWR9
+L GND-RESCUE-12V_Supply #PWR01
 U 1 1 55C54F23
 P 7450 3150
-F 0 "#PWR9" H 7450 3150 30  0001 C CNN
+F 0 "#PWR01" H 7450 3150 30  0001 C CNN
 F 1 "GND" H 7450 3080 30  0001 C CNN
 F 2 "" H 7450 3150 60  0000 C CNN
@@
 $EndComp
 $Comp
-L GND-RESCUE-12V_Supply #PWR2
+L GND-RESCUE-12V_Supply #PWR02
 U 1 1 55C54FA5
 P 7450 2500
-F 0 "#PWR2" H 7450 2500 30  0001 C CNN
+F 0 "#PWR02" H 7450 2500 30  0001 C CNN
 F 1 "GND" H 7450 2430 30  0001 C CNN
 F 2 "" H 7450 2500 60  0000 C CNN
@@
 $EndComp
 $Comp
-L GND-RESCUE-12V_Supply #PWR8
+L GND-RESCUE-12V_Supply #PWR03
 U 1 1 55C54FCF
 P 6550 2600
-F 0 "#PWR8" H 6550 2600 30  0001 C CNN
+F 0 "#PWR03" H 6550 2600 30  0001 C CNN
 F 1 "GND" H 6550 2530 30  0001 C CNN
 F 2 "" H 6550 2600 60  0000 C CNN
@@
 $EndComp
 $Comp
-L GND-RESCUE-12V_Supply #PWR7
+L GND-RESCUE-12V_Supply #PWR04
 U 1 1 55C55002
 P 5750 2600
-F 0 "#PWR7" H 5750 2600 30  0001 C CNN
+F 0 "#PWR04" H 5750 2600 30  0001 C CNN
 F 1 "GND" H 5750 2530 30  0001 C CNN
 F 2 "" H 5750 2600 60  0000 C CNN
@@
 $EndComp
 $Comp
-L GND-RESCUE-12V_Supply #PWR6
+L GND-RESCUE-12V_Supply #PWR05
 U 1 1 55C5507B
 P 5100 2600
-F 0 "#PWR6" H 5100 2600 30  0001 C CNN
+F 0 "#PWR05" H 5100 2600 30  0001 C CNN
 F 1 "GND" H 5100 2530 30  0001 C CNN
 F 2 "" H 5100 2600 60  0000 C CNN
@@
 $EndComp
 $Comp
-L GND-RESCUE-12V_Supply #PWR5
+L GND-RESCUE-12V_Supply #PWR06
 U 1 1 55C550A7
 P 4350 2600
-F 0 "#PWR5" H 4350 2600 30  0001 C CNN
+F 0 "#PWR06" H 4350 2600 30  0001 C CNN
 F 1 "GND" H 4350 2530 30  0001 C CNN
 F 2 "" H 4350 2600 60  0000 C CNN
@@
 $EndComp
 $Comp
-L GND-RESCUE-12V_Supply #PWR4
+L GND-RESCUE-12V_Supply #PWR07
 U 1 1 55C550D3
 P 3650 2600
-F 0 "#PWR4" H 3650 2600 30  0001 C CNN
+F 0 "#PWR07" H 3650 2600 30  0001 C CNN
 F 1 "GND" H 3650 2530 30  0001 C CNN
 F 2 "" H 3650 2600 60  0000 C CNN
@@
 $EndComp
 $Comp
-L GND-RESCUE-12V_Supply #PWR3
+L GND-RESCUE-12V_Supply #PWR08
 U 1 1 55C550FF
 P 2300 2600
-F 0 "#PWR3" H 2300 2600 30  0001 C CNN
+F 0 "#PWR08" H 2300 2600 30  0001 C CNN
 F 1 "GND" H 2300 2530 30  0001 C CNN
 F 2 "" H 2300 2600 60  0000 C CNN
@@
 	7450 2500 7450 2400
 $Comp
-L +12V #PWR1
+L +12V #PWR09
 U 1 1 55C558D9
 P 7150 1950
-F 0 "#PWR1" H 7150 1900 20  0001 C CNN
+F 0 "#PWR09" H 7150 1900 20  0001 C CNN
 F 1 "+12V" H 7150 2050 30  0000 C CNN
 F 2 "" H 7150 1950 60  0000 C CNN
@@
 L D D4
 U 1 1 55C5639B
-P 6850 4650
-F 0 "D4" H 6850 4750 50  0000 C CNN
-F 1 "1N4001" H 6850 4550 50  0000 C CNN
-F 2 "w_pth_diodes:diode_do41" H 6850 4650 60  0001 C CNN
-F 3 "" H 6850 4650 60  0000 C CNN
-	1    6850 4650
-	1    0    0    -1
-$EndComp
-$Comp
-L GND-RESCUE-12V_Supply #PWR13
+P 6550 4650
+F 0 "D4" H 6550 4750 50  0000 C CNN
+F 1 "1N4001" H 6550 4550 50  0000 C CNN
+F 2 "w_pth_diodes:diode_do41" H 6550 4650 60  0001 C CNN
+F 3 "" H 6550 4650 60  0000 C CNN
+	1    6550 4650
+	1    0    0    -1
+$EndComp
+$Comp
+L GND-RESCUE-12V_Supply #PWR010
 U 1 1 55C5698D
 P 5050 5400
-F 0 "#PWR13" H 5050 5400 30  0001 C CNN
+F 0 "#PWR010" H 5050 5400 30  0001 C CNN
 F 1 "GND" H 5050 5330 30  0001 C CNN
 F 2 "" H 5050 5400 60  0000 C CNN
@@
 P 5950 5200
 F 0 "C4" H 5975 5300 50  0000 L CNN
-F 1 "1µF" H 5975 5100 50  0000 L CNN
+F 1 "200µF" H 5975 5100 50  0000 L CNN
 F 2 "w_capacitors:CP_4x5mm" H 5988 5050 30  0001 C CNN
 F 3 "" H 5950 5200 60  0000 C CNN
@@
 P 5950 4050
 F 0 "R1" V 6030 4050 50  0000 C CNN
-F 1 "18k" V 5950 4050 50  0000 C CNN
-F 2 "Resistors_ThroughHole:Resistor_Horizontal_RM10mm" V 5880 4050 30  0001 C CNN
+F 1 "47k" V 5950 4050 50  0000 C CNN
+F 2 "Resistors_THT:R_Axial_DIN0207_L6.3mm_D2.5mm_P10.16mm_Horizontal" V 5880 4050 30  0001 C CNN
 F 3 "" H 5950 4050 30  0000 C CNN
 	1    5950 4050
@@
 Connection ~ 5950 4300
 $Comp
-L GND-RESCUE-12V_Supply #PWR14
+L GND-RESCUE-12V_Supply #PWR011
 U 1 1 55C57D8C
 P 5950 5450
-F 0 "#PWR14" H 5950 5450 30  0001 C CNN
+F 0 "#PWR011" H 5950 5450 30  0001 C CNN
 F 1 "GND" H 5950 5380 30  0001 C CNN
 F 2 "" H 5950 5450 60  0000 C CNN
@@
 NoConn ~ 4350 4900
 Text Notes 3900 4150 0    60   ~ 0
-Power-On-Delay\n20s\n(Tdelay = 1.1 * C * R)
+Power-On-Delay\nca. 10s\n(Tdelay = 1.1 * C * R)
 Connection ~ 7150 2800
 Wire Wire Line
@@
 	5500 4300 5500 4150
 $Comp
-L +12V #PWR11
+L +12V #PWR012
 U 1 1 55C5B443
 P 5050 3750
-F 0 "#PWR11" H 5050 3700 20  0001 C CNN
+F 0 "#PWR012" H 5050 3700 20  0001 C CNN
 F 1 "+12V" H 5050 3850 30  0000 C CNN
 F 2 "" H 5050 3750 60  0000 C CNN
@@
 $EndComp
 Wire Wire Line
-	5950 3900 5950 3800
-Wire Wire Line
-	5950 3800 5050 3800
+	5950 3800 5950 3900
+Wire Wire Line
+	5050 3800 5950 3800
 Connection ~ 5050 3800
 Wire Wire Line
@@
 Connection ~ 5500 4300
 Wire Wire Line
-	5750 4650 6700 4650
-Wire Wire Line
-	7450 4650 7000 4650
+	5750 4650 6400 4650
+Wire Wire Line
+	6700 4650 7450 4650
 Wire Wire Line
 	7150 4450 7450 4450
@@
 F 0 "P5" V 7750 3400 40  0000 C CNN
 F 1 "12V_DC_3" V 7850 3400 40  0000 C CNN
-F 2 "MiniUniversalMate-N-LokSockets_13Aug2012:MiniUniversalMate-N-LokSocket_2PinVertical_12Aug2012" H 7800 3400 60  0001 C CNN
+F 2 "Connectors_Mini-Universal:MiniUniversalMate-N-LokSocket_2PinVertical" H 7800 3400 60  0001 C CNN
 F 3 "" H 7800 3400 60  0000 C CNN
 	1    7800 3400
@@
 	7150 3300 7450 3300
 $Comp
-L GND-RESCUE-12V_Supply #PWR10
+L GND-RESCUE-12V_Supply #PWR013
 U 1 1 55C680B0
 P 7450 3650
-F 0 "#PWR10" H 7450 3650 30  0001 C CNN
+F 0 "#PWR013" H 7450 3650 30  0001 C CNN
 F 1 "GND" H 7450 3580 30  0001 C CNN
 F 2 "" H 7450 3650 60  0000 C CNN
@@
 F 0 "P6" V 7750 3950 40  0000 C CNN
 F 1 "12V_DC_4" V 7850 3950 40  0000 C CNN
-F 2 "MiniUniversalMate-N-LokSockets_13Aug2012:MiniUniversalMate-N-LokSocket_2PinVertical_12Aug2012" H 7800 3950 60  0001 C CNN
+F 2 "Connectors_Mini-Universal:MiniUniversalMate-N-LokSocket_2PinVertical" H 7800 3950 60  0001 C CNN
 F 3 "" H 7800 3950 60  0000 C CNN
 	1    7800 3950
@@
 	7150 3850 7450 3850
 $Comp
-L GND-RESCUE-12V_Supply #PWR12
+L GND-RESCUE-12V_Supply #PWR014
 U 1 1 55C68115
 P 7450 4200
-F 0 "#PWR12" H 7450 4200 30  0001 C CNN
+F 0 "#PWR014" H 7450 4200 30  0001 C CNN
 F 1 "GND" H 7450 4130 30  0001 C CNN
 F 2 "" H 7450 4200 60  0000 C CNN
@@
 	2300 2600 2300 2200
 $Comp
-L PWR_FLAG #FLG1
+L PWR_FLAG #FLG015
 U 1 1 55CDAF94
 P 6900 2200
-F 0 "#FLG1" H 6900 2470 30  0001 C CNN
+F 0 "#FLG015" H 6900 2470 30  0001 C CNN
 F 1 "PWR_FLAG" H 6900 2430 30  0000 C CNN
 F 2 "" H 6900 2200 60  0000 C CNN
@@
 F 0 "R2" V 3330 2200 50  0000 C CNN
 F 1 "10R" V 3250 2200 50  0000 C CNN
-F 2 "Resistors_ThroughHole:Resistor_Horizontal_RM10mm" V 3180 2200 30  0001 C CNN
+F 2 "Resistors_THT:R_Axial_DIN0207_L6.3mm_D2.5mm_P10.16mm_Horizontal" V 3180 2200 30  0001 C CNN
 F 3 "" H 3250 2200 30  0000 C CNN
 	1    3250 2200
@@
 	7300 5050 7450 5050
 Connection ~ 7300 4650
+$Comp
+L LED D5
+U 1 1 5A176B87
+P 6850 4300
+F 0 "D5" H 6850 4400 50  0000 C CNN
+F 1 "LED" H 6850 4200 50  0000 C CNN
+F 2 "LEDs:LED_D3.0mm" H 6850 4300 50  0001 C CNN
+F 3 "" H 6850 4300 50  0001 C CNN
+	1    6850 4300
+	0    -1   -1   0
+$EndComp
+$Comp
+L R R3
+U 1 1 5A176DF9
+P 6850 3900
+F 0 "R3" V 6930 3900 50  0000 C CNN
+F 1 "47k" V 6850 3900 50  0000 C CNN
+F 2 "Resistors_THT:R_Axial_DIN0207_L6.3mm_D2.5mm_P10.16mm_Horizontal" V 6780 3900 30  0001 C CNN
+F 3 "" H 6850 3900 30  0000 C CNN
+	1    6850 3900
+	1    0    0    -1
+$EndComp
+Wire Wire Line
+	6850 4450 6850 4650
+Connection ~ 6850 4650
+Wire Wire Line
+	6850 4050 6850 4150
+$Comp
+L +12V #PWR016
+U 1 1 5A177000
+P 6850 3650
+F 0 "#PWR016" H 6850 3600 20  0001 C CNN
+F 1 "+12V" H 6850 3750 30  0000 C CNN
+F 2 "" H 6850 3650 60  0000 C CNN
+F 3 "" H 6850 3650 60  0000 C CNN
+	1    6850 3650
+	1    0    0    -1
+$EndComp
+Wire Wire Line
+	6850 3750 6850 3650
 $EndSCHEMATC

Commit message: Work in Progress
Parts:
- C1, C4, C5: symbol CP -> Device:CP
- C2, C3: symbol C -> Device:C
- D1: symbol BRIDGE -> w_device:BRIDGE
- D2, D3, D4: symbol D -> Device:D
- D5: symbol LED -> Device:LED
- F1: symbol F_Small -> 12V_Supply-rescue:F_Small
- P1, P2, P3, P4, P5, P6, P7: symbol CONN_2 -> borniers:CONN_2
- R1, R2, R3: symbol R -> Device:R
- TR1: symbol TRANSF1 -> 12V_Supply-rescue:TRANSF1
- U1: symbol LM555N-RESCUE-12V_Supply -> 12V_Supply-rescue:LM555N-RESCUE-12V_Supply
- U2: symbol LM7812CT -> 12V_Supply-rescue:LM7812CT
Changed lines of the file:
@@
-EESchema Schematic File Version 2
-LIBS:12V_Supply-rescue
-LIBS:power
-LIBS:device
-LIBS:transistors
-LIBS:conn
-LIBS:linear
-LIBS:regul
-LIBS:74xx
-LIBS:cmos4000
-LIBS:adc-dac
-LIBS:memory
-LIBS:xilinx
-LIBS:microcontrollers
-LIBS:dsp
-LIBS:microchip
-LIBS:analog_switches
-LIBS:motorola
-LIBS:texas
-LIBS:intel
-LIBS:audio
-LIBS:interface
-LIBS:digital-audio
-LIBS:philips
-LIBS:display
-LIBS:cypress
-LIBS:siliconi
-LIBS:opto
-LIBS:atmel
-LIBS:contrib
-LIBS:valves
-LIBS:w_connectors
-LIBS:w_device
-LIBS:w_transistor
-LIBS:borniers
-LIBS:74xgxx
-LIBS:ac-dc
-LIBS:actel
-LIBS:Altera
-LIBS:analog_devices
-LIBS:brooktre
-LIBS:cmos_ieee
-LIBS:dc-dc
-LIBS:diode
-LIBS:elec-unifil
-LIBS:ESD_Protection
-LIBS:ftdi
-LIBS:gennum
-LIBS:hc11
-LIBS:ir
-LIBS:Lattice
-LIBS:maxim
-LIBS:microchip_dspic33dsc
-LIBS:microchip_pic10mcu
-LIBS:microchip_pic12mcu
-LIBS:microchip_pic16mcu
-LIBS:microchip_pic18mcu
-LIBS:microchip_pic32mcu
-LIBS:motor_drivers
-LIBS:msp430
-LIBS:nordicsemi
-LIBS:nxp_armmcu
-LIBS:onsemi
-LIBS:Oscillators
-LIBS:Power_Management
-LIBS:powerint
-LIBS:pspice
-LIBS:references
-LIBS:relays
-LIBS:rfcom
-LIBS:sensors
-LIBS:silabs
-LIBS:stm8
-LIBS:stm32
-LIBS:supertex
-LIBS:switches
-LIBS:transf
-LIBS:ttl_ieee
-LIBS:video
-LIBS:Xicor
-LIBS:Zilog
+EESchema Schematic File Version 4
 LIBS:12V_Supply-cache
-EELAYER 25 0
+EELAYER 26 0
 EELAYER END
 $Descr A4 11693 8268
@@
 $EndDescr
 $Comp
-L BRIDGE D1
+L w_device:BRIDGE D1
 U 1 1 55C52B4F
 P 2600 2200
@@
 $EndComp
 $Comp
-L CONN_2 P1
+L borniers:CONN_2 P1
 U 1 1 55C544D9
 P 950 2200
@@
 $EndComp
 $Comp
-L LM7812CT U2
+L 12V_Supply-rescue:LM7812CT U2
 U 1 1 55C54685
 P 5100 2250
@@
 $EndComp
 $Comp
-L CP C1
+L Device:CP C1
 U 1 1 55C546E0
 P 3650 2350
@@
 $EndComp
 $Comp
-L C C2
+L Device:C C2
 U 1 1 55C54749
 P 4350 2350
@@
 $EndComp
 $Comp
-L C C3
+L Device:C C3
 U 1 1 55C547E2
 P 5750 2350
@@
 $EndComp
 $Comp
-L CP C5
+L Device:CP C5
 U 1 1 55C5482E
 P 6550 2350
@@
 Connection ~ 4350 2200
 Wire Wire Line
-	5500 2200 7450 2200
+	5500 2200 5750 2200
 Connection ~ 5750 2200
 $Comp
-L CONN_2 P2
+L borniers:CONN_2 P2
 U 1 1 55C54C8E
 P 7800 2300
@@
 $EndComp
 $Comp
-L CONN_2 P3
+L borniers:CONN_2 P3
 U 1 1 55C54D95
 P 7800 2900
@@
 	7150 2800 7450 2800
 Wire Wire Line
-	7150 1950 7150 4850
+	7150 1950 7150 2200
 Connection ~ 7150 2200
 $Comp
-L GND-RESCUE-12V_Supply #PWR01
+L 12V_Supply-rescue:GND-RESCUE-12V_Supply #PWR01
 U 1 1 55C54F23
 P 7450 3150
@@
 $EndComp
 $Comp
-L GND-RESCUE-12V_Supply #PWR02
+L 12V_Supply-rescue:GND-RESCUE-12V_Supply #PWR02
 U 1 1 55C54FA5
 P 7450 2500
@@
 $EndComp
 $Comp
-L GND-RESCUE-12V_Supply #PWR03
+L 12V_Supply-rescue:GND-RESCUE-12V_Supply #PWR03
 U 1 1 55C54FCF
 P 6550 2600
@@
 $EndComp
 $Comp
-L GND-RESCUE-12V_Supply #PWR04
+L 12V_Supply-rescue:GND-RESCUE-12V_Supply #PWR04
 U 1 1 55C55002
 P 5750 2600
@@
 $EndComp
 $Comp
-L GND-RESCUE-12V_Supply #PWR05
+L 12V_Supply-rescue:GND-RESCUE-12V_Supply #PWR05
 U 1 1 55C5507B
 P 5100 2600
@@
 $EndComp
 $Comp
-L GND-RESCUE-12V_Supply #PWR06
+L 12V_Supply-rescue:GND-RESCUE-12V_Supply #PWR06
 U 1 1 55C550A7
 P 4350 2600
@@
 $EndComp
 $Comp
-L GND-RESCUE-12V_Supply #PWR07
+L 12V_Supply-rescue:GND-RESCUE-12V_Supply #PWR07
 U 1 1 55C550D3
 P 3650 2600
@@
 $EndComp
 $Comp
-L GND-RESCUE-12V_Supply #PWR08
+L 12V_Supply-rescue:GND-RESCUE-12V_Supply #PWR08
 U 1 1 55C550FF
 P 2300 2600
@@
 	7450 2500 7450 2400
 $Comp
-L +12V #PWR09
+L power:+12V #PWR09
 U 1 1 55C558D9
 P 7150 1950
@@
 $EndComp
 $Comp
-L LM555N-RESCUE-12V_Supply U1
+L 12V_Supply-rescue:LM555N-RESCUE-12V_Supply U1
 U 1 1 55C55C2A
 P 5050 4850
@@
 $EndComp
 $Comp
-L CONN_2 P4
+L borniers:CONN_2 P4
 U 1 1 55C56025
 P 7800 4550
@@
 $EndComp
 $Comp
-L D D4
+L Device:D D4
 U 1 1 55C5639B
 P 6550 4650
@@
 $EndComp
 $Comp
-L GND-RESCUE-12V_Supply #PWR010
+L 12V_Supply-rescue:GND-RESCUE-12V_Supply #PWR010
 U 1 1 55C5698D
 P 5050 5400
@@
 	5050 5400 5050 5250
 $Comp
-L CP C4
+L Device:CP C4
 U 1 1 55C574DA
 P 5950 5200
@@
 $EndComp
 $Comp
-L R R1
+L Device:R R1
 U 1 1 55C576FC
 P 5950 4050
@@
 $EndComp
 $Comp
-L D D3
+L Device:D D3
 U 1 1 55C578BD
 P 5500 4000
@@
 	5950 5050 5750 5050
 Wire Wire Line
-	5950 4200 5950 5050
+	5950 4200 5950 4300
 Wire Wire Line
 	4350 4650 4300 4650
@@
 Connection ~ 5950 4300
 $Comp
-L GND-RESCUE-12V_Supply #PWR011
+L 12V_Supply-rescue:GND-RESCUE-12V_Supply #PWR011
 U 1 1 55C57D8C
 P 5950 5450
@@
 	5950 5450 5950 5350
 $Comp
-L D D2
+L Device:D D2
 U 1 1 55C58641
 P 5100 1800
@@
 Connection ~ 7150 2800
 Wire Wire Line
-	5050 3750 5050 4450
-Wire Wire Line
-	4300 4300 5950 4300
+	5050 3750 5050 3800
+Wire Wire Line
+	4300 4300 5500 4300
 Wire Wire Line
 	5500 4300 5500 4150
 $Comp
-L +12V #PWR012
+L power:+12V #PWR012
 U 1 1 55C5B443
 P 5050 3750
@@
 	5950 3800 5950 3900
 Wire Wire Line
-	5050 3800 5950 3800
+	5050 3800 5500 3800
 Connection ~ 5050 3800
 Wire Wire Line
@@
 	5750 4650 6400 4650
 Wire Wire Line
-	6700 4650 7450 4650
+	6700 4650 6850 4650
 Wire Wire Line
 	7150 4450 7450 4450
@@
 Connection ~ 5500 2200
 $Comp
-L F_Small F1
+L 12V_Supply-rescue:F_Small F1
 U 1 1 55C5D9C9
 P 2250 1900
@@
 	2350 1900 2600 1900
 $Comp
-L CONN_2 P5
+L borniers:CONN_2 P5
 U 1 1 55C680A8
 P 7800 3400
@@
 	7150 3300 7450 3300
 $Comp
-L GND-RESCUE-12V_Supply #PWR013
+L 12V_Supply-rescue:GND-RESCUE-12V_Supply #PWR013
 U 1 1 55C680B0
 P 7450 3650
@@
 	7450 3500 7450 3650
 $Comp
-L CONN_2 P6
+L borniers:CONN_2 P6
 U 1 1 55C6810E
 P 7800 3950
@@
 	7150 3850 7450 3850
 $Comp
-L GND-RESCUE-12V_Supply #PWR014
+L 12V_Supply-rescue:GND-RESCUE-12V_Supply #PWR014
 U 1 1 55C68115
 P 7450 4200
@@
 	2300 2600 2300 2200
 $Comp
-L PWR_FLAG #FLG015
+L power:PWR_FLAG #FLG015
 U 1 1 55CDAF94
 P 6900 2200
@@
 Connection ~ 6900 2200
 $Comp
-L TRANSF1 TR1
+L 12V_Supply-rescue:TRANSF1 TR1
 U 1 1 55CD0FFE
 P 1750 2200
@@
 $EndComp
 $Comp
-L R R2
+L Device:R R2
 U 1 1 55D87104
 P 3250 2200
@@
 	2900 2200 3100 2200
 Wire Wire Line
-	4700 2200 3400 2200
-$Comp
-L CONN_2 P7
+	4700 2200 4350 2200
+$Comp
+L borniers:CONN_2 P7
 U 1 1 55DE74EC
 P 7800 4950
@@
 Connection ~ 7300 4650
 $Comp
-L LED D5
+L Device:LED D5
 U 1 1 5A176B87
 P 6850 4300
@@
 $EndComp
 $Comp
-L R R3
+L Device:R R3
 U 1 1 5A176DF9
 P 6850 3900
@@
 	6850 4050 6850 4150
 $Comp
-L +12V #PWR016
+L power:+12V #PWR016
 U 1 1 5A177000
 P 6850 3650
@@
 Wire Wire Line
 	6850 3750 6850 3650
+Wire Wire Line
+	3650 2200 3400 2200
+Wire Wire Line
+	4350 2200 3650 2200
+Wire Wire Line
+	5750 2200 6550 2200
+Wire Wire Line
+	6550 2200 6900 2200
+Wire Wire Line
+	7150 2200 7150 2800
+Wire Wire Line
+	7150 2200 7450 2200
+Wire Wire Line
+	5950 4300 5950 5050
+Wire Wire Line
+	7150 2800 7150 3300
+Wire Wire Line
+	5050 3800 5050 4450
+Wire Wire Line
+	5500 3800 5950 3800
+Wire Wire Line
+	5500 4300 5950 4300
+Wire Wire Line
+	7150 3300 7150 3850
+Wire Wire Line
+	7150 3850 7150 4450
+Wire Wire Line
+	6900 2200 7150 2200
+Wire Wire Line
+	7150 4450 7150 4850
+Wire Wire Line
+	7300 4650 7450 4650
+Wire Wire Line
+	6850 4650 7300 4650
 $EndSCHEMATC
