File: Boards/Endstufe/Endstufe.sch (KiCad schematic (older format))
At the start: 74 parts, among them P1 CONN_3, P2 Trafo, P3 Relais, P4 6V3_AC, P5 Trafo_GK, P6 6V3_DC, P7 CONN_4, Q1 2SC2979, Q2 MJE5731, T1 KT88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

Commit message: Anoden-Stabi auf eigenes Board, Endstufe Layouttest
Parts:
- removed C14, C19: 10µF/400V, Capacitors_Elko_ThroughHole:Elko_vert_25x12.5mm_RM5, symbol CP
- removed C15, C17, C20: 47µF/400V, Capacitors_Elko_ThroughHole:Elko_vert_31.5x16mm_RM7.5, symbol CP
- removed C16, C18, C21: 1µF/400V, Capacitors_ThroughHole:C_Rect_L32_W15_P27, symbol C
- removed D1, D2: BZT03-C150, Diodes_ThroughHole:Diode_DO-41_SOD81_Horizontal_RM10, symbol ZENER
- removed D3: BZT03-C120, Diodes_ThroughHole:Diode_DO-41_SOD81_Horizontal_RM10, symbol ZENER
- removed P7: CONN_4, MiniUniversalMate-N-LokSockets_13Aug2012:MiniUniversalMate-N-LokSocket_4PinVertical_13Aug2012, symbol CONN_4
- removed Q1: 2SC2979, w_to:to220-horiz_5772, symbol Q_NPN_BCE
- removed Q2: MJE5731, w_to:to220-horiz_5772, symbol Q_PNP_BCE
- removed R24: 82k, Resistors_ThroughHole:Resistor_Horizontal_RM10mm, symbol R
- removed R25: 10k/1W, Resistors_ThroughHole:Resistor_Horizontal_RM15mm, symbol R
- removed R26, R28, R30: 1k5, Resistors_ThroughHole:Resistor_Horizontal_RM10mm, symbol R
- removed R27: 33k, Resistors_ThroughHole:Resistor_Horizontal_RM10mm, symbol R
- removed R29, R31: 30k, Resistors_ThroughHole:Resistor_Horizontal_RM10mm, symbol R
- added P7: VSup1, Sockets_Mini-Universal:MiniUniversalMate-N-LokSocket_2PinVertical, symbol CONN_2
- added P8: Vsup2, Sockets_Mini-Universal:MiniUniversalMate-N-LokSocket_2PinVertical, symbol CONN_2
- added P9: VSup3, Sockets_Mini-Universal:MiniUniversalMate-N-LokSocket_4PinVertical, symbol CONN_4
- C11, C2, C4, C8: footprint Capacitors_ThroughHole:C_Rect_L18_W5_P15 -> w_capacitors:CPA_8x21MM
- C7: footprint Capacitors_ThroughHole:C_Disc_D6_P5 -> w_capacitors:CPA_8x21MM
- P2: footprint (none) -> Sockets_WAGO734:WAGO_734_5pin_Straight
- P4, P5, P6: footprint MiniUniversalMate-N-LokSockets_13Aug2012:MiniUniversalMate-N-LokSocket_2PinVertical_12Aug2012 -> Sockets_Mini-Universal:MiniUniversalMate-N-LokSocket_2PinVertical
Connections:
- net labels removed: -180V
- wire segments 195 -> 157
Other:
- note added: "Mallory 150's 0,1 µF / 630 VDC"
- moved on the sheet: C1, C10, C11, C12, C13, C2, C3, C4, C5, C6, C7, C8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

Commit message: Layouting...
Parts:
- removed P8: Vsup2, Sockets_Mini-Universal:MiniUniversalMate-N-LokSocket_2PinVertical, symbol CONN_2
- added R24: 30k, Resistors_ThroughHole:Resistor_Horizontal_RM10mm, symbol R
Connections:
- wire segments 157 -> 155
Changed lines of the file:
@@
 $EndComp
 $Comp
-L GND #PWR01
+L GND #PWR1
 U 1 1 55C91E71
 P 1050 2450
-F 0 "#PWR01" H 1050 2200 50  0001 C CNN
+F 0 "#PWR1" H 1050 2200 50  0001 C CNN
 F 1 "GND" H 1050 2300 50  0000 C CNN
 F 2 "" H 1050 2450 60  0000 C CNN
@@
 $EndComp
 $Comp
-L GND #PWR02
+L GND #PWR6
 U 1 1 55C9279C
 P 5100 2000
-F 0 "#PWR02" H 5100 1750 50  0001 C CNN
+F 0 "#PWR6" H 5100 1750 50  0001 C CNN
 F 1 "GND" H 5100 1850 50  0000 C CNN
 F 2 "" H 5100 2000 60  0000 C CNN
@@
 $EndComp
 $Comp
-L GND #PWR03
+L GND #PWR7
 U 1 1 55C92CDE
 P 5100 4350
-F 0 "#PWR03" H 5100 4100 50  0001 C CNN
+F 0 "#PWR7" H 5100 4100 50  0001 C CNN
 F 1 "GND" H 5100 4200 50  0000 C CNN
 F 2 "" H 5100 4350 60  0000 C CNN
@@
 $EndComp
 $Comp
-L GND #PWR04
+L GND #PWR10
 U 1 1 55C96A98
 P 9450 2750
-F 0 "#PWR04" H 9450 2500 50  0001 C CNN
+F 0 "#PWR10" H 9450 2500 50  0001 C CNN
 F 1 "GND" H 9450 2600 50  0000 C CNN
 F 2 "" H 9450 2750 60  0000 C CNN
@@
 $EndComp
 $Comp
-L GND #PWR05
+L GND #PWR8
 U 1 1 55C999B3
 P 7100 2850
-F 0 "#PWR05" H 7100 2600 50  0001 C CNN
+F 0 "#PWR8" H 7100 2600 50  0001 C CNN
 F 1 "GND" H 7100 2700 50  0000 C CNN
 F 2 "" H 7100 2850 60  0000 C CNN
@@
 $EndComp
 $Comp
-L GND #PWR06
+L GND #PWR4
 U 1 1 55CA0096
 P 2150 2800
-F 0 "#PWR06" H 2150 2550 50  0001 C CNN
+F 0 "#PWR4" H 2150 2550 50  0001 C CNN
 F 1 "GND" H 2150 2650 50  0000 C CNN
 F 2 "" H 2150 2800 60  0000 C CNN
@@
 $EndComp
 $Comp
-L GND #PWR07
+L GND #PWR11
 U 1 1 55CA27EB
 P 10150 3400
-F 0 "#PWR07" H 10150 3150 50  0001 C CNN
+F 0 "#PWR11" H 10150 3150 50  0001 C CNN
 F 1 "GND" H 10150 3250 50  0000 C CNN
 F 2 "" H 10150 3400 60  0000 C CNN
@@
 6V3
 $Comp
-L PWR_FLAG #FLG08
+L PWR_FLAG #FLG1
 U 1 1 55CC6FF3
 P 7550 6000
-F 0 "#FLG08" H 7550 6095 50  0001 C CNN
+F 0 "#FLG1" H 7550 6095 50  0001 C CNN
 F 1 "PWR_FLAG" H 7550 6180 50  0000 C CNN
 F 2 "" H 7550 6000 60  0000 C CNN
@@
 $EndComp
 $Comp
-L GND #PWR09
+L GND #PWR12
 U 1 1 55CDF4D0
 P 10900 4350
-F 0 "#PWR09" H 10900 4100 50  0001 C CNN
+F 0 "#PWR12" H 10900 4100 50  0001 C CNN
 F 1 "GND" H 10900 4200 50  0000 C CNN
 F 2 "" H 10900 4350 60  0000 C CNN
@@
 $EndComp
 $Comp
-L GND #PWR010
+L GND #PWR9
 U 1 1 55D03168
 P 8450 2900
-F 0 "#PWR010" H 8450 2650 50  0001 C CNN
+F 0 "#PWR9" H 8450 2650 50  0001 C CNN
 F 1 "GND" H 8450 2750 50  0000 C CNN
 F 2 "" H 8450 2900 60  0000 C CNN
@@
 $EndComp
 $Comp
-L PWR_FLAG #FLG011
+L PWR_FLAG #FLG2
 U 1 1 55D3787B
 P 8900 6200
-F 0 "#FLG011" H 8900 6295 50  0001 C CNN
+F 0 "#FLG2" H 8900 6295 50  0001 C CNN
 F 1 "PWR_FLAG" H 8900 6380 50  0000 C CNN
 F 2 "" H 8900 6200 60  0000 C CNN
@@
 $EndComp
 $Comp
-L GND #PWR012
+L GND #PWR3
 U 1 1 55DB93E3
 P 1550 3750
-F 0 "#PWR012" H 1550 3500 50  0001 C CNN
+F 0 "#PWR3" H 1550 3500 50  0001 C CNN
 F 1 "GND" H 1550 3600 50  0000 C CNN
 F 2 "" H 1550 3750 60  0000 C CNN
@@
 $EndComp
 $Comp
-L CONN_2 P8
-U 1 1 56BBDDEA
-P 900 6550
-F 0 "P8" V 850 6550 40  0000 C CNN
-F 1 "Vsup2" V 950 6550 40  0000 C CNN
-F 2 "Sockets_Mini-Universal:MiniUniversalMate-N-LokSocket_2PinVertical" H 900 6550 60  0001 C CNN
-F 3 "" H 900 6550 60  0000 C CNN
-	1    900  6550
-	-1   0    0    -1
-$EndComp
-$Comp
-L GND #PWR013
-U 1 1 56BBEC8D
-P 1350 6700
-F 0 "#PWR013" H 1350 6450 50  0001 C CNN
-F 1 "GND" H 1350 6550 50  0000 C CNN
-F 2 "" H 1350 6700 60  0000 C CNN
-F 3 "" H 1350 6700 60  0000 C CNN
-	1    1350 6700
-	1    0    0    -1
-$EndComp
-$Comp
-L GND #PWR014
+L GND #PWR2
 U 1 1 56BBED46
 P 1400 5900
-F 0 "#PWR014" H 1400 5650 50  0001 C CNN
+F 0 "#PWR2" H 1400 5650 50  0001 C CNN
 F 1 "GND" H 1400 5750 50  0000 C CNN
 F 2 "" H 1400 5900 60  0000 C CNN
@@
 Text GLabel 1650 5650 2    60   Input ~ 0
 +450V
-Text GLabel 1650 6450 2    60   Input ~ 0
+Text GLabel 3550 6100 2    60   Input ~ 0
 -60V
 $Comp
@@
 	1250 5650 1650 5650
 Wire Wire Line
-	1250 6450 1650 6450
-Wire Wire Line
 	1250 5850 1400 5850
 Wire Wire Line
 	1400 5850 1400 5900
-Wire Wire Line
-	1250 6650 1350 6650
-Wire Wire Line
-	1350 6650 1350 6700
-$Comp
-L GND #PWR015
+$Comp
+L GND #PWR5
 U 1 1 56BC14D7
 P 3050 5950
-F 0 "#PWR015" H 3050 5700 50  0001 C CNN
+F 0 "#PWR5" H 3050 5700 50  0001 C CNN
 F 1 "GND" H 3050 5800 50  0000 C CNN
 F 2 "" H 3050 5950 60  0000 C CNN
@@
 	3050 5900 3050 5950
 Wire Wire Line
-	2900 5800 3150 5800
-Wire Wire Line
-	2900 5700 3550 5700
-Wire Wire Line
-	2900 5600 3900 5600
-Text GLabel 3900 5600 2    60   Input ~ 0
+	2900 5800 3550 5800
+Wire Wire Line
+	2900 5700 3900 5700
+Wire Wire Line
+	2900 5600 4250 5600
+Text GLabel 4250 5600 2    60   Input ~ 0
 +300V
-Text GLabel 3550 5700 2    60   Input ~ 0
+Text GLabel 3900 5700 2    60   Input ~ 0
 +240V
-Text GLabel 3150 5800 2    60   Input ~ 0
+Text GLabel 3550 5800 2    60   Input ~ 0
 -120V
+$Comp
+L R R24
+U 1 1 56C095ED
+P 3350 5950
+F 0 "R24" V 3430 5950 50  0000 C CNN
+F 1 "30k" V 3350 5950 50  0000 C CNN
+F 2 "Resistors_ThroughHole:Resistor_Horizontal_RM10mm" V 3280 5950 30  0001 C CNN
+F 3 "" H 3350 5950 30  0000 C CNN
+	1    3350 5950
+	-1   0    0    1
+$EndComp
+Wire Wire Line
+	3350 6100 3550 6100
+Connection ~ 3350 5800
 $EndSCHEMATC

Commit message: Updated Layout
Connections:
- wire segments 155 -> 204
Changed lines of the file:
@@
 	1    0    0    -1
 $EndComp
-Text GLabel 1650 5650 2    60   Input ~ 0
+Text GLabel 1400 5650 2    60   Input ~ 0
 +450V
 Text GLabel 3550 6100 2    60   Input ~ 0
@@
 $EndComp
 Wire Wire Line
-	3350 2550 3350 2950
-Wire Wire Line
-	5450 2000 5450 3550
+	3350 2550 3350 2700
+Wire Wire Line
+	3350 2700 3350 2950
+Wire Wire Line
+	5450 2000 5450 2700
+Wire Wire Line
+	5450 2700 5450 3550
 Wire Wire Line
 	3250 2700 3350 2700
@@
 	3450 1750 3450 1600
 Wire Wire Line
-	3450 1600 4650 1600
-Wire Wire Line
-	4950 1600 5250 1600
+	3450 1600 4200 1600
+Wire Wire Line
+	4200 1600 4550 1600
+Wire Wire Line
+	4550 1600 4650 1600
+Wire Wire Line
+	4950 1600 5100 1600
+Wire Wire Line
+	5100 1600 5250 1600
 Connection ~ 5100 1600
 Wire Wire Line
 	5100 1900 5100 2000
 Wire Wire Line
-	4900 3950 5250 3950
+	4900 3950 5100 3950
+Wire Wire Line
+	5100 3950 5250 3950
 Connection ~ 5100 3950
 Wire Wire Line
-	3450 3950 4600 3950
+	3450 3950 4200 3950
+Wire Wire Line
+	4200 3950 4550 3950
+Wire Wire Line
+	4550 3950 4600 3950
 Wire Wire Line
 	3450 3950 3450 3750
@@
 	5550 4500 6100 4500
 Wire Wire Line
-	6100 4500 6100 3400
-Wire Wire Line
-	6100 2300 6100 3100
-Wire Wire Line
-	6100 1100 6100 2000
+	6100 4500 6100 4000
+Wire Wire Line
+	6100 4000 6100 3400
+Wire Wire Line
+	6100 2300 6100 2700
+Wire Wire Line
+	6100 2700 6100 3100
+Wire Wire Line
+	6100 1100 6100 1650
+Wire Wire Line
+	6100 1650 6100 2000
 Connection ~ 6100 2700
 Wire Wire Line
@@
 	5550 1100 6100 1100
 Wire Wire Line
-	6550 4000 8150 4000
+	6550 4000 7600 4000
+Wire Wire Line
+	7600 4000 7800 4000
+Wire Wire Line
+	7800 4000 7900 4000
+Wire Wire Line
+	7900 4000 8150 4000
 Wire Wire Line
 	6250 4000 6100 4000
 Connection ~ 6100 4000
 Wire Wire Line
-	6550 1650 8150 1650
+	6550 1650 7600 1650
+Wire Wire Line
+	7600 1650 7800 1650
+Wire Wire Line
+	7800 1650 7900 1650
+Wire Wire Line
+	7900 1650 8150 1650
 Wire Wire Line
 	6250 1650 6100 1650
 Connection ~ 6100 1650
 Wire Wire Line
-	8750 1700 9600 1700
+	8750 1700 9000 1700
+Wire Wire Line
+	9000 1700 9600 1700
 Wire Wire Line
 	9600 1700 9600 2100
 Wire Wire Line
-	9600 2400 9600 3200
+	9600 2400 9600 2700
+Wire Wire Line
+	9600 2700 9600 3200
 Wire Wire Line
 	9450 2750 9450 2700
@@
 Connection ~ 7600 1650
 Wire Wire Line
-	8750 3950 9600 3950
+	8750 3950 9000 3950
+Wire Wire Line
+	9000 3950 9600 3950
 Wire Wire Line
 	9600 3950 9600 3500
 Wire Wire Line
-	1000 2150 3150 2150
+	1000 2150 1650 2150
+Wire Wire Line
+	1650 2150 2350 2150
+Wire Wire Line
+	2350 2150 3150 2150
 Wire Wire Line
 	2350 2200 2350 2150
 Connection ~ 2350 2150
 Wire Wire Line
-	2350 2500 2350 3000
+	2350 2500 2350 2700
+Wire Wire Line
+	2350 2700 2350 3000
 Wire Wire Line
 	2150 2800 2150 2700
@@
 Connection ~ 2350 2700
 Wire Wire Line
-	2350 3300 2350 4650
+	2350 3300 2350 3350
+Wire Wire Line
+	2350 3350 2350 4650
 Wire Wire Line
 	2350 4650 10400 4650
@@
 	10550 4450 10550 4400
 Wire Wire Line
-	10250 4450 10550 4450
+	10250 4450 10400 4450
+Wire Wire Line
+	10400 4450 10550 4450
 Wire Wire Line
 	10250 4450 10250 4300
@@
 	10150 3300 10150 3400
 Wire Wire Line
-	10400 4650 10400 4150
+	10400 4650 10400 4450
+Wire Wire Line
+	10400 4450 10400 4150
 Wire Wire Line
 	10550 3850 10550 3900
@@
 	10250 4000 10250 3850
 Wire Wire Line
-	10250 3850 10550 3850
+	10250 3850 10400 3850
+Wire Wire Line
+	10400 3850 10550 3850
 Wire Wire Line
 	8650 6000 8650 5950
@@
 	10550 3500 10400 3500
 Wire Wire Line
-	10400 3500 10400 3850
+	10400 3500 10400 3650
+Wire Wire Line
+	10400 3650 10400 3850
 Connection ~ 10400 3850
 Wire Wire Line
@@
 Connection ~ 7800 1650
 Wire Wire Line
-	7500 2100 7800 2100
+	7500 2100 7600 2100
+Wire Wire Line
+	7600 2100 7800 2100
 Wire Wire Line
 	7800 2100 7800 2000
 Wire Wire Line
-	7600 2050 7600 2200
+	7600 2050 7600 2100
+Wire Wire Line
+	7600 2100 7600 2200
 Connection ~ 7600 2100
 Wire Wire Line
 	7350 2350 7350 2400
 Wire Wire Line
-	7350 2700 7350 2900
+	7350 2700 7350 2800
+Wire Wire Line
+	7350 2800 7350 2900
 Wire Wire Line
 	7350 3250 7350 3200
@@
 Connection ~ 7350 2800
 Wire Wire Line
-	7600 3450 7600 3600
-Wire Wire Line
-	7500 3500 7800 3500
+	7600 3450 7600 3500
+Wire Wire Line
+	7600 3500 7600 3600
+Wire Wire Line
+	7500 3500 7600 3500
+Wire Wire Line
+	7600 3500 7800 3500
 Connection ~ 7600 3500
 Wire Wire Line
 	7800 3500 7800 3600
 Wire Wire Line
-	7600 2500 7600 3150
+	7600 2500 7600 2700
+Wire Wire Line
+	7600 2700 7600 3150
 Wire Wire Line
 	7650 2700 7600 2700
@@
 	2850 2700 2950 2700
 Wire Wire Line
-	8200 1800 8200 3850
-Wire Wire Line
-	8700 1800 8700 3850
+	8200 1800 8200 2700
+Wire Wire Line
+	8200 2700 8200 3250
+Wire Wire Line
+	8200 3250 8200 3850
+Wire Wire Line
+	8700 1800 8700 2700
+Wire Wire Line
+	8700 2700 8700 3450
+Wire Wire Line
+	8700 3450 8700 3850
 Connection ~ 8200 2700
 Connection ~ 8700 2700
@@
 Connection ~ 8200 3250
 Wire Wire Line
-	1650 2150 1650 2450
+	1650 2150 1650 2400
+Wire Wire Line
+	1650 2400 1650 2450
 Connection ~ 1650 2150
 Wire Wire Line
-	1650 2750 1650 2950
+	1650 2750 1650 2800
+Wire Wire Line
+	1650 2800 1650 2950
 Wire Wire Line
 	1450 2450 1450 2400
@@
 	1450 2750 1450 2800
 Wire Wire Line
-	1450 2800 1900 2800
+	1450 2800 1650 2800
+Wire Wire Line
+	1650 2800 2000 2800
 Connection ~ 1650 2800
 Wire Wire Line
 	1750 3550 1750 3600
 Wire Wire Line
-	1750 3600 1900 3600
-Wire Wire Line
-	1900 3600 1900 2800
+	1750 3600 2000 3600
+Wire Wire Line
+	2000 3600 2000 2800
 Wire Wire Line
 	1550 3550 1550 3750
@@
 	950  3550 950  3350
 Wire Wire Line
-	7450 6000 8650 6000
-Wire Wire Line
-	7450 6200 8900 6200
+	7450 6000 7550 6000
+Wire Wire Line
+	7550 6000 7750 6000
+Wire Wire Line
+	7750 6000 7950 6000
+Wire Wire Line
+	7950 6000 8450 6000
+Wire Wire Line
+	8450 6000 8650 6000
+Wire Wire Line
+	7450 6200 7850 6200
+Wire Wire Line
+	7850 6200 8550 6200
+Wire Wire Line
+	8550 6200 8900 6200
 Wire Wire Line
 	8550 6200 8550 5950
@@
 	1000 2350 1050 2350
 Wire Wire Line
-	1050 2250 1050 2450
+	1050 2250 1050 2350
+Wire Wire Line
+	1050 2350 1050 2450
 Wire Wire Line
 	1000 2250 1050 2250
@@
 	2750 4950 2800 4950
 Wire Wire Line
-	1250 5650 1650 5650
+	1250 5650 1400 5650
 Wire Wire Line
 	1250 5850 1400 5850
@@
 	3050 5900 3050 5950
 Wire Wire Line
-	2900 5800 3550 5800
-Wire Wire Line
-	2900 5700 3900 5700
-Wire Wire Line
-	2900 5600 4250 5600
-Text GLabel 4250 5600 2    60   Input ~ 0
+	2900 5800 3350 5800
+Wire Wire Line
+	3350 5800 3550 5800
+Wire Wire Line
+	2900 5700 3950 5700
+Wire Wire Line
+	2900 5600 4350 5600
+Text GLabel 4350 5600 2    60   Input ~ 0
 +300V
-Text GLabel 3900 5700 2    60   Input ~ 0
+Text GLabel 3950 5700 2    60   Input ~ 0
 +240V
 Text GLabel 3550 5800 2    60   Input ~ 0

Commit message: Work in Progress
Parts:
- RV1, RV2, RV3, RV4, RV5: symbol POT -> POT-RESCUE-Endstufe
Connections:
- wire segments 204 -> 155
Changed lines of the file:
@@
 EESchema Schematic File Version 2
+LIBS:Endstufe-rescue
 LIBS:power
 LIBS:device
@@
 $EndComp
 $Comp
-L POT RV2
+L POT-RESCUE-Endstufe RV2
 U 1 1 55C91BEC
 P 4200 2700
@@
 $EndComp
 $Comp
-L POT RV1
+L POT-RESCUE-Endstufe RV1
 U 1 1 55C981AE
 P 7350 2100
@@
 $EndComp
 $Comp
-L POT RV4
+L POT-RESCUE-Endstufe RV4
 U 1 1 55C989D7
 P 7350 3500
@@
 $EndComp
 $Comp
-L POT RV5
+L POT-RESCUE-Endstufe RV5
 U 1 1 55CA2532
 P 10550 4150
@@
 -120V
 $Comp
-L POT RV3
+L POT-RESCUE-Endstufe RV3
 U 1 1 55D01699
 P 8450 2700
@@
 $EndComp
 Wire Wire Line
-	3350 2550 3350 2700
-Wire Wire Line
-	3350 2700 3350 2950
-Wire Wire Line
-	5450 2000 5450 2700
-Wire Wire Line
-	5450 2700 5450 3550
+	3350 2550 3350 2950
+Wire Wire Line
+	5450 2000 5450 3550
 Wire Wire Line
 	3250 2700 3350 2700
@@
 	3450 1750 3450 1600
 Wire Wire Line
-	3450 1600 4200 1600
-Wire Wire Line
-	4200 1600 4550 1600
-Wire Wire Line
-	4550 1600 4650 1600
-Wire Wire Line
-	4950 1600 5100 1600
-Wire Wire Line
-	5100 1600 5250 1600
+	3450 1600 4650 1600
+Wire Wire Line
+	4950 1600 5250 1600
 Connection ~ 5100 1600
 Wire Wire Line
 	5100 1900 5100 2000
 Wire Wire Line
-	4900 3950 5100 3950
-Wire Wire Line
-	5100 3950 5250 3950
+	4900 3950 5250 3950
 Connection ~ 5100 3950
 Wire Wire Line
-	3450 3950 4200 3950
-Wire Wire Line
-	4200 3950 4550 3950
-Wire Wire Line
-	4550 3950 4600 3950
+	3450 3950 4600 3950
 Wire Wire Line
 	3450 3950 3450 3750
@@
 	5550 4350 5550 4500
 Wire Wire Line
-	5550 4500 6100 4500
-Wire Wire Line
-	6100 4500 6100 4000
-Wire Wire Line
-	6100 4000 6100 3400
-Wire Wire Line
-	6100 2300 6100 2700
-Wire Wire Line
-	6100 2700 6100 3100
-Wire Wire Line
-	6100 1100 6100 1650
-Wire Wire Line
-	6100 1650 6100 2000
+	6100 4500 5550 4500
+Wire Wire Line
+	6100 3400 6100 4500
+Wire Wire Line
+	6100 2300 6100 3100
+Wire Wire Line
+	6100 1100 6100 2000
 Connection ~ 6100 2700
 Wire Wire Line
@@
 	5550 1100 6100 1100
 Wire Wire Line
-	6550 4000 7600 4000
-Wire Wire Line
-	7600 4000 7800 4000
-Wire Wire Line
-	7800 4000 7900 4000
-Wire Wire Line
-	7900 4000 8150 4000
+	6550 4000 8150 4000
 Wire Wire Line
 	6250 4000 6100 4000
 Connection ~ 6100 4000
 Wire Wire Line
-	6550 1650 7600 1650
-Wire Wire Line
-	7600 1650 7800 1650
-Wire Wire Line
-	7800 1650 7900 1650
-Wire Wire Line
-	7900 1650 8150 1650
+	6550 1650 8150 1650
 Wire Wire Line
 	6250 1650 6100 1650
 Connection ~ 6100 1650
 Wire Wire Line
-	8750 1700 9000 1700
-Wire Wire Line
-	9000 1700 9600 1700
+	8750 1700 9600 1700
 Wire Wire Line
 	9600 1700 9600 2100
 Wire Wire Line
-	9600 2400 9600 2700
-Wire Wire Line
-	9600 2700 9600 3200
+	9600 2400 9600 3200
 Wire Wire Line
 	9450 2750 9450 2700
@@
 Connection ~ 7600 1650
 Wire Wire Line
-	8750 3950 9000 3950
-Wire Wire Line
-	9000 3950 9600 3950
+	8750 3950 9600 3950
 Wire Wire Line
 	9600 3950 9600 3500
 Wire Wire Line
-	1000 2150 1650 2150
-Wire Wire Line
-	1650 2150 2350 2150
-Wire Wire Line
-	2350 2150 3150 2150
+	1000 2150 3150 2150
 Wire Wire Line
 	2350 2200 2350 2150
 Connection ~ 2350 2150
 Wire Wire Line
-	2350 2500 2350 2700
-Wire Wire Line
-	2350 2700 2350 3000
+	2350 2500 2350 3000
 Wire Wire Line
 	2150 2800 2150 2700
@@
 Connection ~ 2350 2700
 Wire Wire Line
-	2350 3300 2350 3350
-Wire Wire Line
-	2350 3350 2350 4650
-Wire Wire Line
-	2350 4650 10400 4650
+	2350 3300 2350 4650
+Wire Wire Line
+	10400 4650 2350 4650
 Wire Wire Line
 	2350 3350 3150 3350
@@
 	10550 4450 10550 4400
 Wire Wire Line
-	10250 4450 10400 4450
-Wire Wire Line
-	10400 4450 10550 4450
+	10250 4450 10550 4450
 Wire Wire Line
 	10250 4450 10250 4300
@@
 	10150 3300 10150 3400
 Wire Wire Line
-	10400 4650 10400 4450
-Wire Wire Line
-	10400 4450 10400 4150
+	10400 4150 10400 4650
 Wire Wire Line
 	10550 3850 10550 3900
@@
 	10250 4000 10250 3850
 Wire Wire Line
-	10250 3850 10400 3850
-Wire Wire Line
-	10400 3850 10550 3850
+	10250 3850 10550 3850
 Wire Wire Line
 	8650 6000 8650 5950
@@
 	10550 3500 10400 3500
 Wire Wire Line
-	10400 3500 10400 3650
-Wire Wire Line
-	10400 3650 10400 3850
+	10400 3500 10400 3850
 Connection ~ 10400 3850
 Wire Wire Line
@@
 Connection ~ 7800 1650
 Wire Wire Line
-	7500 2100 7600 2100
-Wire Wire Line
-	7600 2100 7800 2100
+	7500 2100 7800 2100
 Wire Wire Line
 	7800 2100 7800 2000
 Wire Wire Line
-	7600 2050 7600 2100
-Wire Wire Line
-	7600 2100 7600 2200
+	7600 2050 7600 2200
 Connection ~ 7600 2100
 Wire Wire Line
 	7350 2350 7350 2400
 Wire Wire Line
-	7350 2700 7350 2800
-Wire Wire Line
-	7350 2800 7350 2900
+	7350 2700 7350 2900
 Wire Wire Line
 	7350 3250 7350 3200
@@
 Connection ~ 7350 2800
 Wire Wire Line
-	7600 3450 7600 3500
-Wire Wire Line
-	7600 3500 7600 3600
-Wire Wire Line
-	7500 3500 7600 3500
-Wire Wire Line
-	7600 3500 7800 3500
+	7600 3450 7600 3600
+Wire Wire Line
+	7500 3500 7800 3500
 Connection ~ 7600 3500
 Wire Wire Line
 	7800 3500 7800 3600
 Wire Wire Line
-	7600 2500 7600 2700
-Wire Wire Line
-	7600 2700 7600 3150
+	7600 2500 7600 3150
 Wire Wire Line
 	7650 2700 7600 2700
@@
 	2850 2700 2950 2700
 Wire Wire Line
-	8200 1800 8200 2700
-Wire Wire Line
-	8200 2700 8200 3250
-Wire Wire Line
-	8200 3250 8200 3850
-Wire Wire Line
-	8700 1800 8700 2700
-Wire Wire Line
-	8700 2700 8700 3450
-Wire Wire Line
-	8700 3450 8700 3850
+	8200 1800 8200 3850
+Wire Wire Line
+	8700 1800 8700 3850
 Connection ~ 8200 2700
 Connection ~ 8700 2700
@@
 Connection ~ 8200 3250
 Wire Wire Line
-	1650 2150 1650 2400
-Wire Wire Line
-	1650 2400 1650 2450
+	1650 2150 1650 2450
 Connection ~ 1650 2150
 Wire Wire Line
-	1650 2750 1650 2800
-Wire Wire Line
-	1650 2800 1650 2950
+	1650 2750 1650 2950
 Wire Wire Line
 	1450 2450 1450 2400
@@
 	1450 2750 1450 2800
 Wire Wire Line
-	1450 2800 1650 2800
-Wire Wire Line
-	1650 2800 2000 2800
+	1450 2800 2000 2800
 Connection ~ 1650 2800
 Wire Wire Line
@@
 	950  3550 950  3350
 Wire Wire Line
-	7450 6000 7550 6000
-Wire Wire Line
-	7550 6000 7750 6000
-Wire Wire Line
-	7750 6000 7950 6000
-Wire Wire Line
-	7950 6000 8450 6000
-Wire Wire Line
-	8450 6000 8650 6000
-Wire Wire Line
-	7450 6200 7850 6200
-Wire Wire Line
-	7850 6200 8550 6200
-Wire Wire Line
-	8550 6200 8900 6200
+	7450 6000 8650 6000
+Wire Wire Line
+	7450 6200 8900 6200
 Wire Wire Line
 	8550 6200 8550 5950
@@
 	1000 2350 1050 2350
 Wire Wire Line
-	1050 2250 1050 2350
-Wire Wire Line
-	1050 2350 1050 2450
+	1050 2250 1050 2450
 Wire Wire Line
 	1000 2250 1050 2250
@@
 	3050 5900 3050 5950
 Wire Wire Line
-	2900 5800 3350 5800
-Wire Wire Line
-	3350 5800 3550 5800
+	2900 5800 3550 5800
 Wire Wire Line
 	2900 5700 3950 5700

Commit message: Work in Progress
Parts:
- removed P9: VSup3, Sockets_Mini-Universal:MiniUniversalMate-N-LokSocket_4PinVertical, symbol CONN_4
- removed RL1: FINDER-36.11.4001, w_relay:relay_34.51, symbol FINDER-36.11.4001
- removed RV1, RV4: 10k, w_pth_resistors:trimmer_piher_pt6xv, symbol POT-RESCUE-Endstufe
- added C14, C15: 10µF / 100V, Capacitors_ThroughHole:C_Radial_D6.3_L11.2_P2.5, symbol C_Small
- added K1: DIP 7212-D, Reed:REED, symbol DIP~7212-D
- added P8: Bias, Pin_Headers:Pin_Header_Straight_2x03_Pitch2.54mm, symbol CONN_01X06
- added P9: CONN_5, symbol CONN_5
- C1, C13, C5, C9: value 68pF -> 68pF / 500V; footprint Capacitor-Wima-FKP2-630v:Capacitor-Wima-FKP2-630v-R5B4K5 -> Capacitors_ThroughHole:C_Disc_D7.5_P5
- C10, C3: value 100nF -> 100nF / 400V; footprint Capacitors_ThroughHole:C_Rect_L7.5_W6.5_P5 -> Capacitors_ThroughHole:C_Axial_D8_L21_P28
- C11, C2, C4, C8: value 100nF/630V -> 100nF/400V; footprint w_capacitors:CPA_8x21MM -> Capacitors_ThroughHole:C_Axial_D8_L21_P28
- C12: value 100pF -> 100pF / 500V; footprint Capacitors_ThroughHole:C_Disc_D3_P2.5 -> Capacitors_ThroughHole:C_Disc_D7.5_P5
- C6: value 33pF -> 33pF / 500V
- C7: value 100nF/630V -> 100nF; footprint w_capacitors:CPA_8x21MM -> Capacitors_ThroughHole:C_Disc_D3_P2.5
- R10, R13, R20, R23, R5: footprint Resistors_ThroughHole:Resistor_Horizontal_RM20mm -> Resistors_ThroughHole:Resistor_Ceramic_Horizontal_L23mm-W9mm-H9mm-p30mm
- R9: value 68k -> 220R
- RV2, RV3, RV5: footprint w_pth_resistors:trimmer_piher_pt6xv -> w_pth_resistors:trimmer_piher_pt10xv10
Connections:
- net labels added: Bias_1, Bias_2, UG_1, UG_2
- wire segments 155 -> 158
Other:
- note added: "Ausgang / Übertrager"
- note added: "ECC83 Vorstufe"
- note added: "Eingang / Knackunterdrückung"
- note added: "Gegenkopplung"
- note added: "Glimmer"
- note added: "Heizung ECC83"
- note added: "KT88 Endstufe"
- note added: "Roederstein MKT 1813\n400 V DC"
- note removed: "Mallory 150's 0,1 µF / 630 VDC"
- moved on the sheet: C7, P4, P7, R20, R5, R9
