File: Boards/Endstufe/Endstufe.kicad_pcb (KiCad board)
At the start: 2 copper layers, 165 x 130 mm, 62 parts, among them J1 HV In, J10 240V VU, J2 Relais, J3 Audio_In, J4 Übertrager, J5 Gegenkopplung, J6 12V out, J7 Conn_01x08, J8 12V In, J9 VU-Meter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

Commit message: Leiterplatte erstellt
Parts:
- removed the G*** at (53.0, 50.3)
- removed K1: G6E, Relay_THT:Relay_SPDT_Omron_G6E
- removed REF**: Symbol_HighVoltage_Type2_SilkTop_VerySmall, Loewe:Symbol_HighVoltage_Type2_SilkTop_VerySmall
- added H1: MountingHole, MountingHole:MountingHole_3.2mm_M3, F.Cu at (202.8, 166.3)
- added H2: MountingHole, MountingHole:MountingHole_3.2mm_M3, F.Cu at (202.8, 46.3)
- added H3: MountingHole, MountingHole:MountingHole_3.2mm_M3, F.Cu at (57.8, 46.3)
- added H4: MountingHole, MountingHole:MountingHole_3.2mm_M3, F.Cu at (57.8, 166.3)
- added H5: MountingHole, MountingHole:MountingHole_3.2mm_M3, F.Cu at (111.2, 106.3)
- added H6: MountingHole, MountingHole:MountingHole_3.2mm_M3, F.Cu at (177.2, 106.3)
- added K2: G5V-1, Relay_THT:Relay_SPDT_Omron_G5V-1, F.Cu at (55.2, 89.0)
- C1, C12, C13, C5, C9: footprint Capacitor_THT:C_Disc_D7.5mm_W4.4mm_P5.00mm -> Capacitor_THT:C_Disc_D11.0mm_W5.0mm_P7.50mm
- C10, C11, C2, C3, C4, C7, C8: footprint Capacitor_THT:C_Axial_L22.0mm_D9.5mm_P27.50mm_Horizontal -> Capacitor_THT:C_Axial_L19.0mm_D7.5mm_P25.00mm_Horizontal
- C14, C15: value 10µF/100V -> 10µF/400V; footprint Capacitor_THT:CP_Radial_D6.3mm_P2.50mm -> Capacitor_THT:CP_Radial_D10.0mm_P5.00mm
- C6: footprint Capacitor_THT:C_Disc_D6.0mm_W4.4mm_P5.00mm -> Capacitor_THT:C_Disc_D11.0mm_W5.0mm_P7.50mm
- J1: footprint Connector_TE-Connectivity:TE_MATE-N-LOK_1-770875-x_2x03_P4.14mm_Vertical -> Connector_Molex:Molex_Mini-Fit_Jr_5566-06A_2x03_P4.20mm_Vertical
- J10, J5, J9, P1, P2, P6: footprint Connector_TE-Connectivity:TE_MATE-N-LOK_1-770866-x_1x02_P4.14mm_Vertical -> Connector_Molex:Molex_Mini-Fit_Jr_5566-02A_2x01_P4.20mm_Vertical
- J4: footprint Connector_TE-Connectivity:TE_MATE-N-LOK_350211-1_1x04_P5.08mm_Vertical -> Connector_Molex:Molex_Mini-Fit_Jr_5566-04A_2x02_P4.20mm_Vertical
- RV2, RV5: footprint Potentiometer_THT:Potentiometer_Piher_PT-10-V10_Vertical_Hole -> Potentiometer_THT:Potentiometer_Vishay_T7-YA_Single_Vertical; moved to B.Cu
- T1, T2: footprint Valve:Valve_Octal -> ValveSockets:Valve_Octal
- U1, U2: footprint Valve:Valve_ECC-83-1 -> ValveSockets:Valve_Noval
- moved P1 21.7 mm to (181.6, 42.4), turned to -90 degrees
- moved T1 13.0 mm to (177.2, 63.8)
- moved P6 12.7 mm to (111.3, 121.4)
- moved G*** 12.3 mm to (142.0, 158.0)
- moved R9 9.79 mm to (57.4, 105.2)
- moved T2 9.67 mm to (177.2, 148.8)
- moved RV5 9.31 mm to (84.2, 133.3), turned to 90 degrees
- moved J2 8.36 mm to (61.5, 71.9), turned to 180 degrees
- moved C1 7.63 mm to (156.0, 52.3)
- moved U1 6.32 mm to (132.2, 106.3)
- moved J10 5.95 mm to (71.6, 56.9)
- moved RV2 5.89 mm to (84.2, 79.3), turned to -90 degrees
- moved U2 5.49 mm to (90.2, 106.3)
- moved C15 5.39 mm to (143.4, 133.0), turned to 90 degrees
- moved J4 5.24 mm to (199.1, 95.8), turned to 0 degrees
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Connections:
- C11 pad 1: Net-(C11-Pad1) -> Net-(T2-g1)
- C13 pad 1: Bias_2 -> Net-(T2-g1)
- C13 pad 2: Net-(C11-Pad1) -> Bias_2
- C14 pad 1: Net-(C14-Pad1) -> GND
- C14 pad 2: GND -> Net-(C14-Pad2)
- C15 pad 1: Net-(C15-Pad1) -> GND
- C15 pad 2: GND -> Net-(C15-Pad2)
- C5 pad 1: Net-(C14-Pad1) -> Net-(C14-Pad2)
- C8 pad 1: Net-(C11-Pad1) -> Net-(T2-g1)
- C9 pad 1: Net-(C11-Pad1) -> Net-(T2-g1)
- C9 pad 2: Net-(C15-Pad1) -> Net-(C15-Pad2)
- J1 pad 1: GND -> -120V
- J1 pad 2: -120V -> -60V
- J1 pad 3: +300V -> GND
- J1 pad 4: +240V -> GND
- J1 pad 5: GND -> +240V
- J1 pad 6: -60V -> +300V
- R14 pad 1: Net-(C15-Pad1) -> Net-(C15-Pad2)
- R17 pad 1: Net-(C15-Pad1) -> Net-(C15-Pad2)
- R2 pad 1: Net-(C14-Pad1) -> Net-(C14-Pad2)
- R21 pad 1: Net-(C11-Pad1) -> Net-(T2-g1)
- R21 pad 2: Net-(C15-Pad1) -> Net-(C15-Pad2)
- R7 pad 2: Net-(C14-Pad1) -> Net-(C14-Pad2)
- R8 pad 1: Net-(C14-Pad1) -> Net-(C14-Pad2)
- T2 pad 5: Net-(C11-Pad1) -> Net-(T2-g1)
Routing:
- net Net-(C11-Pad1): track 51.3 -> 0.00 mm
- net Net-(T2-g1): track 0.00 -> 49.9 mm
- net Net-(P6-P2): track 52.6 -> 80.9 mm
- net Net-(C14-Pad2): track 0.00 -> 24.8 mm
- net Net-(C15-Pad1): track 22.7 -> 0.00 mm
- net Net-(P1-P1): track 50.2 -> 27.7 mm
- net Net-(C15-Pad2): track 0.00 -> 20.9 mm
- net -120V: track 53.2 -> 73.5 mm
- net Net-(C14-Pad1): track 18.4 -> 0.00 mm
- net Net-(J5-Pin_1): track 45.5 -> 28.2 mm
- net +240V: track 41.3 -> 55.5 mm
- net /+450V_T1: track 61.2 -> 47.1 mm
- net Net-(U2A-K): track 27.8 -> 40.8 mm
- net Net-(J4-Pin_4): track 15.7 -> 28.6 mm
- net Net-(U1A-K): track 27.9 -> 40.6 mm
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Other:
- board size 165 x 130 mm -> 165 x 135 mm
- rule pad_to_mask_clearance: 0.2 -> 0
- board text added: "D. Walter v1.1"
- board text removed: "D. Walter v1.0"
- board text removed: "HIGH VOLTAGE!"
