File: Boards/Netzteil/400V_Anoden/400VAnoden.kicad_pcb (KiCad board)
At the start: 2 copper layers, 44 parts, among them P1 Drossel, P2 450V_AC, P3 CONN_4, P4 -120V_AC, P5 CONN_4, Q1 2SC2979

Commit message: Anoden-Stabi auf eigenes Board, Endstufe Layouttest
Parts:
- added REF**: EuroBoard160mmX100mm_holes, EuroBoard_Outline:EuroBoard160mmX100mm_holes, F.Cu at (36.6, 127.0)
Other:
- board outline added: 160 x 100 mm
Changed lines of the file:
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@@
-(kicad_pcb (version 4) (host pcbnew "(2015-08-21 BZR 6112, Git 0386a4d)-product")
+(kicad_pcb (version 4) (host pcbnew 4.0.1-stable)
   (general
-    (links 70)
+    (links 0)
     (no_connects 0)
     (area 36.068 25.908 212.344001 134.620001)
@@
     (tracks 152)
     (zones 0)
-    (modules 44)
+    (modules 45)
     (nets 24)
   )
@@
   )
   (setup
-    (last_trace_width 1)
+    (last_trace_width 0.5)
     (user_trace_width 0.5)
     (user_trace_width 1)
@@
     (pad "" np_thru_hole circle (at 6.52018 -2.0701 270) (size 3.2004 3.2004) (drill 3.2004) (layers *.Cu *.Mask F.SilkS))
   )
+  (module EuroBoard_Outline:EuroBoard160mmX100mm_holes (layer F.Cu)
+    (at 36.576 127)
+    (descr "Outline, Eurocard, 100x160mm, with holes 3,5mm,")
+    (tags "Outline, Eurocard, 100x160mm, with holes 3,5mm,")
+    (fp_text reference REF** (at 78.74 -60.96) (layer F.SilkS)
+      (effects (font (size 1 1) (thickness 0.15)))
+    )
+    (fp_text value EuroBoard160mmX100mm_holes (at 85.09 -35.56) (layer F.Fab)
+      (effects (font (size 1 1) (thickness 0.15)))
+    )
+    (fp_line (start 1.00076 -99.9998) (end 0 -99.9998) (layer F.SilkS) (width 0.15))
+    (fp_line (start 0 -99.9998) (end 0 0) (layer Edge.Cuts) (width 0.381))
+    (fp_line (start 0 0) (end 159.99968 0) (layer Edge.Cuts) (width 0.381))
+    (fp_line (start 159.99968 0) (end 159.99968 -99.9998) (layer Edge.Cuts) (width 0.381))
+    (fp_line (start 159.99968 -99.9998) (end 1.00076 -99.9998) (layer Edge.Cuts) (width 0.381))
+    (pad "" np_thru_hole circle (at 5.00126 -95.00108) (size 3.50012 3.50012) (drill 3.50012) (layers *.Cu *.Mask F.SilkS))
+    (pad "" np_thru_hole circle (at 155.00096 -95.00108) (size 3.50012 3.50012) (drill 3.50012) (layers *.Cu *.Mask F.SilkS))
+    (pad "" np_thru_hole circle (at 155.00096 -5.00126) (size 3.50012 3.50012) (drill 3.50012) (layers *.Cu *.Mask F.SilkS))
+    (pad "" np_thru_hole circle (at 5.00126 -5.00126) (size 3.50012 3.50012) (drill 3.50012) (layers *.Cu *.Mask F.SilkS))
+  )
   (segment (start 82.5119 33.528) (end 82.5119 39.4081) (width 1) (layer B.Cu) (net 1) (status 10))
   (segment (start 78.359 43.561) (end 69.977 43.561) (width 1) (layer B.Cu) (net 1) (status 20))
@@
   (segment (start 100.156 58.42) (end 100.076 58.34) (width 0.25) (layer B.Cu) (net 5) (status 30))
   (segment (start 100.076 75.772) (end 100.584 76.28) (width 0.25) (layer B.Cu) (net 5) (status 30))
-  (segment (start 200.9521 65.3161) (end 196.8119 61.1759) (width 1) (layer B.Cu) (net 6) (status C00000))
-  (segment (start 200.6981 84.8741) (end 196.5579 80.7339) (width 1) (layer B.Cu) (net 6) (status C00000))
+  (segment (start 200.9521 65.3161) (end 196.8119 61.1759) (width 1) (layer B.Cu) (net 6))
+  (segment (start 200.6981 84.8741) (end 196.5579 80.7339) (width 1) (layer B.Cu) (net 6))
   (segment (start 101.172 86.868) (end 100.584 86.28) (width 0.25) (layer B.Cu) (net 6) (status 30))
   (segment (start 166.116 87.376) (end 178.816 87.376) (width 1) (layer B.Cu) (net 7) (status 10))
@@
   (segment (start 45.70984 36.07816) (end 48.26 33.528) (width 1) (layer B.Cu) (net 19))
   (segment (start 186.944 75.184) (end 186.944 59.2201) (width 1) (layer B.Cu) (net 20))
-  (segment (start 186.944 59.2201) (end 181.356 53.6321) (width 1) (layer B.Cu) (net 20) (status 800000))
-  (segment (start 196.5579 84.8741) (end 196.5579 86.9061) (width 1) (layer B.Cu) (net 20) (status 400000))
-  (segment (start 186.944 75.184) (end 196.8119 65.3161) (width 1) (layer B.Cu) (net 20) (status 800000))
+  (segment (start 186.944 59.2201) (end 181.356 53.6321) (width 1) (layer B.Cu) (net 20))
+  (segment (start 196.5579 84.8741) (end 196.5579 86.9061) (width 1) (layer B.Cu) (net 20))
+  (segment (start 186.944 75.184) (end 196.8119 65.3161) (width 1) (layer B.Cu) (net 20))
   (segment (start 186.944 86.36) (end 186.944 75.184) (width 1) (layer B.Cu) (net 20))
   (segment (start 190.5 89.916) (end 186.944 86.36) (width 1) (layer B.Cu) (net 20))
@@
   (segment (start 45.98416 118.62816) (end 45.98416 104.4321) (width 1) (layer B.Cu) (net 21) (status 20))
   (segment (start 51.308 123.952) (end 45.98416 118.62816) (width 1) (layer B.Cu) (net 21))
-  (segment (start 200.9521 61.1759) (end 200.9521 51.6001) (width 1) (layer B.Cu) (net 22) (status 400000))
-  (segment (start 167.8559 53.6321) (end 161.798 53.6321) (width 1) (layer B.Cu) (net 22) (status 800000))
+  (segment (start 200.9521 61.1759) (end 200.9521 51.6001) (width 1) (layer B.Cu) (net 22))
+  (segment (start 167.8559 53.6321) (end 161.798 53.6321) (width 1) (layer B.Cu) (net 22))
   (segment (start 173.736 47.752) (end 167.8559 53.6321) (width 1) (layer B.Cu) (net 22))
   (segment (start 197.104 47.752) (end 173.736 47.752) (width 1) (layer B.Cu) (net 22))
   (segment (start 200.9521 51.6001) (end 197.104 47.752) (width 1) (layer B.Cu) (net 22))
-  (segment (start 200.6981 80.7339) (end 203.2381 80.7339) (width 1) (layer B.Cu) (net 22) (status 400000))
-  (segment (start 206.756 66.9798) (end 200.9521 61.1759) (width 1) (layer B.Cu) (net 22) (status 800000))
+  (segment (start 200.6981 80.7339) (end 203.2381 80.7339) (width 1) (layer B.Cu) (net 22))
+  (segment (start 206.756 66.9798) (end 200.9521 61.1759) (width 1) (layer B.Cu) (net 22))
   (segment (start 206.756 77.216) (end 206.756 66.9798) (width 1) (layer B.Cu) (net 22))
   (segment (start 203.2381 80.7339) (end 206.756 77.216) (width 1) (layer B.Cu) (net 22))

Commit message: Updated Layout
Parts:
- removed REF**: EuroBoard160mmX100mm_holes, EuroBoard_Outline:EuroBoard160mmX100mm_holes
- moved F3 28.5 mm to (95.9, 109.9), turned to 180 degrees
- moved R2 25.9 mm to (84.5, 64.8)
- moved R5 18.7 mm to (108.0, 64.8), turned to 270 degrees
- moved D6 18.3 mm to (184.2, 36.8), turned to 0 degrees
- moved P3 13.2 mm to (188.0, 55.9), turned to 90 degrees
- moved P5 12.8 mm to (187.3, 76.8), turned to 270 degrees
- moved F2 7.37 mm to (174.0, 64.8)
- moved R6 5.11 mm to (158.1, 88.3)
- moved C9 4.66 mm to (95.9, 78.7)
- moved C3 4.60 mm to (95.9, 51.4)
- moved R3 4.60 mm to (158.1, 83.8)
- moved C6 4.51 mm to (177.2, 105.4)
- moved C13 3.81 mm to (112.4, 104.1)
- moved C14 3.18 mm to (130.2, 74.3)
- moved C5 2.29 mm to (130.2, 55.9)
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Routing:
- net Net-(F3-Pad1): track 30.7 -> 63.7 mm
- net Net-(F4-Pad2): track 78.7 -> 55.1 mm
- net Net-(C3-Pad1): track 94.7 -> 72.6 mm
- net GND: track 12.5 -> 0.00 mm
- net Net-(F2-Pad2): track 63.4 -> 52.6 mm
- net Net-(C5-Pad1): track 208.5 -> 199.2 mm
- net Net-(D6-Pad2): track 4.42 -> 12.0 mm
- net Net-(C13-Pad2): track 97.7 -> 91.8 mm
- net Net-(C1-Pad1): track 62.1 -> 66.4 mm
- net Net-(C7-Pad2): track 73.1 -> 76.9 mm
- net Net-(C10-Pad1): track 56.0 -> 58.3 mm
- net Net-(C3-Pad2): track 42.2 -> 44.0 mm
Other:
- board outline removed

Commit message: Work in Progress
Parts:
- removed F2: 1AT, w_misc_comp:fuse_holder_CQ-2
- removed F4: F_Small, w_misc_comp:fuse_holder_CQ-2
- added REF**: EuroBoard160mmX100mm_holes, EuroBoard_Outline:EuroBoard160mmX100mm_holes, F.Cu at (36.8, 127.0)
- P2: value 450V_AC -> 320V_AC
- P3, P5: value CONN_4 -> CONN_3; footprint MiniUniversalMate-N-LokSockets_13Aug2012:MiniUniversalMate-N-LokSocket_4PinVertical_13Aug2012 -> Connectors_Mini-Universal:MiniUniversalMate-N-LokSocket_3PinVertical
- P4: value -120V_AC -> 133V_AC
- moved R7 19.4 mm to (171.4, 50.8)
- moved P3 16.5 mm to (188.6, 72.4)
- moved D6 14.0 mm to (183.5, 50.8), turned to 180 degrees
- moved P5 13.5 mm to (174.6, 72.4), turned to 90 degrees
Connections:
- C13 pad 2: Net-(C13-Pad2) -> /-180V_DC
- C14 pad 1: Net-(C13-Pad2) -> /-180V_DC
- C5 pad 1: Net-(C5-Pad1) -> /+450V_DC
- C6 pad 1: Net-(C5-Pad1) -> /+450V_DC
- P1 pad 2: Net-(C5-Pad1) -> /+450V_DC
- P3 pad 1: Net-(F2-Pad2) -> /+450V_DC
- P3 pad 3: GND -> /-180V_DC
- P5 pad 1: Net-(F2-Pad2) -> /+450V_DC
- P5 pad 3: GND -> /-180V_DC
- Q1 pad 2: Net-(C5-Pad1) -> /+450V_DC
- R3 pad 2: Net-(C5-Pad1) -> /+450V_DC
- R4 pad 2: Net-(C5-Pad1) -> /+450V_DC
- R8 pad 1: Net-(C13-Pad2) -> /-180V_DC
Routing:
- net /+450V_DC: track 0.00 -> 225.8 mm, vias 0 -> 2
- net Net-(C5-Pad1): track 199.2 -> 0.00 mm
- net /-180V_DC: track 0.00 -> 121.6 mm
- net Net-(C13-Pad2): track 91.8 -> 0.00 mm
- net Net-(F4-Pad2): track 55.1 -> 0.00 mm
- net Net-(F2-Pad2): track 52.6 -> 0.00 mm
- net Net-(Q1-Pad3): track 33.5 -> 23.6 mm
- net Net-(D6-Pad2): track 12.0 -> 4.44 mm
Other:
- board outline added: 160 x 100 mm

Commit message: Work in Progress
Routing:
- net /+450V_DC: track 225.8 -> 232.2 mm
- net Net-(F1-Pad1): track 40.4 -> 37.2 mm
Other:
- board text added: "Bot"
- board text added: "D. Walter v1.0"
Changed lines of the file:
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@@
     (area 36.08 26.309699 197.520181 128.4866)
     (thickness 1.6)
-    (drawings 0)
-    (tracks 141)
+    (drawings 2)
+    (tracks 142)
     (zones 0)
     (modules 43)
@@
       (outputformat 1)
       (mirror false)
-      (drillshape 1)
+      (drillshape 0)
       (scaleselection 1)
       (outputdirectory ""))
@@
       (net 21 /-180V_DC))
   )
+  (gr_text "D. Walter\nv1.0" (at 187.706 40.386) (layer B.Cu)
+    (effects (font (size 1.5 1.5) (thickness 0.3)) (justify mirror))
+  )
+  (gr_text Bot (at 178.562 122.174) (layer B.Cu)
+    (effects (font (size 1.5 1.5) (thickness 0.3)) (justify mirror))
+  )
   (segment (start 61.976 52.832) (end 61.976 47.033756) (width 1) (layer B.Cu) (net 1))
   (segment (start 61.976 47.033756) (end 58.249244 43.307) (width 1) (layer B.Cu) (net 1))
@@
   (segment (start 70.104 58.674) (end 69.977 58.547) (width 1) (layer B.Cu) (net 2) (status 30))
   (segment (start 54.356 68.707) (end 54.356 58.293) (width 1) (layer B.Cu) (net 3) (status 30))
+  (segment (start 95.885 46.435) (end 95.885 41.83713) (width 1) (layer B.Cu) (net 4))
+  (segment (start 95.885 41.83713) (end 97.7519 39.97023) (width 1) (layer B.Cu) (net 4))
+  (segment (start 97.7519 39.97023) (end 97.7519 33.79216) (width 1) (layer B.Cu) (net 4))
   (segment (start 116.459 37.465) (end 116.459 40.662603) (width 1) (layer B.Cu) (net 4))
   (segment (start 116.459 40.662603) (end 110.686603 46.435) (width 1) (layer B.Cu) (net 4))
@@
   (segment (start 80.137 64.008) (end 84.455 59.69) (width 1) (layer B.Cu) (net 4))
   (segment (start 95.885 46.435) (end 95.885 46.99) (width 1) (layer B.Cu) (net 4))
-  (segment (start 95.885 46.435) (end 95.885 35.65906) (width 1) (layer B.Cu) (net 4))
-  (segment (start 95.885 35.65906) (end 97.7519 33.79216) (width 1) (layer B.Cu) (net 4))
   (segment (start 95.885 73.74) (end 104.06 73.74) (width 1) (layer B.Cu) (net 5))
   (segment (start 104.06 73.74) (end 107.95 69.85) (width 1) (layer B.Cu) (net 5))
@@
   (segment (start 65.024 64.008) (end 65.024 60.96) (width 1) (layer B.Cu) (net 13) (status 10))
   (segment (start 65.024 60.96) (end 61.976 57.912) (width 1) (layer B.Cu) (net 13) (status 20))
-  (segment (start 155.7528 40.64) (end 155.7528 45.6692) (width 1) (layer B.Cu) (net 14) (status 10))
-  (segment (start 155.7528 45.6692) (end 149.352 52.07) (width 1) (layer B.Cu) (net 14) (status 20))
+  (segment (start 155.7528 40.64) (end 155.7528 43.890581) (width 1) (layer B.Cu) (net 14))
+  (segment (start 155.7528 43.890581) (end 149.352 50.291381) (width 1) (layer B.Cu) (net 14))
+  (segment (start 149.352 50.291381) (end 149.352 52.07) (width 1) (layer B.Cu) (net 14))
   (segment (start 149.352 56.388) (end 149.352 52.07) (width 1) (layer B.Cu) (net 14) (status 30))
   (segment (start 176.53 50.8) (end 180.975 50.8) (width 1) (layer B.Cu) (net 15))
@@
   (segment (start 75.184 98.552) (end 73.66 100.076) (width 1) (layer B.Cu) (net 16))
   (segment (start 64.516 100.076) (end 73.66 100.076) (width 1) (layer B.Cu) (net 16) (status 30))
-  (segment (start 45.70984 60.4139) (end 45.70984 36.07816) (width 1) (layer B.Cu) (net 17) (status 10))
-  (segment (start 48.26 33.528) (end 60.7441 33.528) (width 1) (layer B.Cu) (net 17) (status 20))
-  (segment (start 45.70984 36.07816) (end 48.26 33.528) (width 1) (layer B.Cu) (net 17))
+  (segment (start 45.70984 60.4139) (end 45.70984 41.623793) (width 1) (layer B.Cu) (net 17))
+  (segment (start 45.70984 41.623793) (end 53.805633 33.528) (width 1) (layer B.Cu) (net 17))
+  (segment (start 53.805633 33.528) (end 60.7441 33.528) (width 1) (layer B.Cu) (net 17))
   (segment (start 95.885 120.7389) (end 50.2539 120.7389) (width 1) (layer B.Cu) (net 18))
   (segment (start 45.98416 116.46916) (end 45.98416 104.4321) (width 1) (layer B.Cu) (net 18))
   (segment (start 50.2539 120.7389) (end 45.98416 116.46916) (width 1) (layer B.Cu) (net 18))
-  (segment (start 166.37 50.8) (end 166.37 47.625) (width 1) (layer B.Cu) (net 19))
-  (segment (start 166.37 47.625) (end 165.1 46.355) (width 1) (layer B.Cu) (net 19))
-  (segment (start 165.1 46.355) (end 165.1 38.1) (width 1) (layer B.Cu) (net 19))
-  (segment (start 165.1 38.1) (end 162.56 35.56) (width 1) (layer B.Cu) (net 19))
+  (segment (start 166.37 50.8) (end 166.37 39.37) (width 1) (layer B.Cu) (net 19))
+  (segment (start 166.37 39.37) (end 162.56 35.56) (width 1) (layer B.Cu) (net 19))
   (segment (start 162.56 35.56) (end 155.7528 35.56) (width 1) (layer B.Cu) (net 19))
-  (segment (start 183.515 92.075) (end 183.515 81.6102) (width 1) (layer B.Cu) (net 20))
-  (segment (start 183.515 81.6102) (end 188.595 76.5302) (width 1) (layer B.Cu) (net 20))
+  (segment (start 153.2128 38.1) (end 158.935075 38.1) (width 1) (layer B.Cu) (net 20))
+  (segment (start 158.935075 38.1) (end 161.544 40.708925) (width 1) (layer B.Cu) (net 20))
+  (segment (start 161.544 40.708925) (end 161.544 60.332333) (width 1) (layer B.Cu) (net 20))
+  (segment (start 161.544 60.332333) (end 155.328333 66.548) (width 1) (layer B.Cu) (net 20))
+  (segment (start 155.328333 66.548) (end 149.352 66.548) (width 1) (layer B.Cu) (net 20))
+  (segment (start 183.515 92.075) (end 183.515 78.69852) (width 1) (layer B.Cu) (net 20))
+  (segment (start 183.515 78.69852) (end 185.68332 76.5302) (width 1) (layer B.Cu) (net 20))
+  (segment (start 185.68332 76.5302) (end 188.595 76.5302) (width 1) (layer B.Cu) (net 20))
+  (segment (start 183.515 92.075) (end 183.515 88.15945) (width 1) (layer B.Cu) (net 20))
+  (segment (start 183.515 88.15945) (end 179.17555 83.82) (width 1) (layer B.Cu) (net 20))
+  (segment (start 179.17555 83.82) (end 163.195 83.82) (width 1) (layer B.Cu) (net 20))
+  (segment (start 143.891 55.88) (end 143.891 63.937816) (width 1) (layer B.Cu) (net 20))
+  (segment (start 143.891 63.937816) (end 146.501184 66.548) (width 1) (layer B.Cu) (net 20))
+  (segment (start 146.501184 66.548) (end 149.352 66.548) (width 1) (layer B.Cu) (net 20))
   (segment (start 188.595 76.5302) (end 186.827686 76.5302) (width 1) (layer B.Cu) (net 20))
   (segment (start 186.827686 76.5302) (end 174.625 76.5302) (width 1) (layer B.Cu) (net 20))
@@
   (segment (start 179.785 110.41) (end 183.515 106.68) (width 1) (layer B.Cu) (net 20))
   (segment (start 183.515 106.68) (end 183.515 92.075) (width 1) (layer B.Cu) (net 20))
-  (segment (start 183.515 92.075) (end 175.26 83.82) (width 1) (layer B.Cu) (net 20))
-  (segment (start 175.26 83.82) (end 163.195 83.82) (width 1) (layer B.Cu) (net 20))
   (segment (start 101.8921 33.782) (end 101.8921 36.401159) (width 1) (layer B.Cu) (net 20))
   (segment (start 101.8921 36.401159) (end 103.219799 37.728858) (width 1) (layer B.Cu) (net 20))
@@
   (segment (start 114.269942 32.99629) (end 128.24629 32.99629) (width 1) (layer B.Cu) (net 20))
   (segment (start 128.24629 32.99629) (end 143.891 48.641) (width 1) (layer B.Cu) (net 20))
-  (segment (start 153.2128 38.1) (end 160.528 38.1) (width 1) (layer B.Cu) (net 20))
-  (segment (start 154.94 64.008) (end 152.4 66.548) (width 1) (layer B.Cu) (net 20))
-  (segment (start 160.528 38.1) (end 161.544 39.116) (width 1) (layer B.Cu) (net 20))
-  (segment (start 161.544 39.116) (end 161.544 45.895528) (width 1) (layer B.Cu) (net 20))
-  (segment (start 161.544 45.895528) (end 154.94 52.499528) (width 1) (layer B.Cu) (net 20))
-  (segment (start 154.94 52.499528) (end 154.94 64.008) (width 1) (layer B.Cu) (net 20))
-  (segment (start 143.891 55.88) (end 143.891 61.087) (width 1) (layer B.Cu) (net 20))
-  (segment (start 143.891 61.087) (end 149.352 66.548) (width 1) (layer B.Cu) (net 20))
-  (segment (start 149.352 66.548) (end 152.4 66.548) (width 1) (layer B.Cu) (net 20) (status 10))
   (segment (start 116.459 74.295) (end 134.022478 74.295) (width 1) (layer B.Cu) (net 21))
   (segment (start 134.022478 74.295) (end 139.828053 80.100575) (width 1) (layer B.Cu) (net 21))
