File: boards/Aussteuerung/Aussteuerung.kicad_pcb (KiCad board)
At the start: 2 copper layers, 100 x 40 mm, 18 parts, among them J1 6V3_Heater, J2 Signal_R, J3 Signal_R, J4 250VDC, K1 FINDER-34.51, U1 EM84

Commit message: Update
Routing:
- net Net-(D3-Pad1): track 25.2 -> 23.7 mm
- net Net-(D1-Pad2): track 20.7 -> 19.3 mm
- net Net-(R8-Pad2): track 34.3 -> 33.5 mm
- net Net-(J1-Pad1): track 18.5 -> 17.8 mm
- net GND: vias 0 -> 19
Other:
- net class Default removed
