File: boards/Eingang/Eingang.kicad_pcb (KiCad board)
At the start: 2 copper layers, 47.5 x 38.7 mm, 9 parts, among them J1 Out, J2 In_L1, J3 In_R1, J4 Out, J5 In_R2, J6 In_L2

Commit message: Update
Routing:
- net Earth_Clean: vias 6 -> 23
Other:
- net class Default removed
