File: boards/Netzteil/6V3_AC_Distribution/6V3_AC_Distribution.kicad_pcb (KiCad board)
At the start: 2 copper layers, 80 x 25 mm, 7 parts, among them J1 Conn_01x02, J2 Conn_01x02, J3 Conn_01x02, J4 Conn_01x02, J6 Screw_Terminal_01x01

Commit message: Update
Other:
- net class Default removed
