File: boards/NoLoad_Protection/Protection/Protection.kicad_pcb (KiCad board)
At the start: 2 copper layers, 80 x 50 mm, 29 parts, among them J1 Transformer, J3 12V_In, J4 Standby, J5 Speaker, J6 Feedback, K1 FINDER-32.21-x000, Q1 BC546, Q2 BC327, Q3 BC337

Commit message: Update
Parts:
- removed D4: 1N4148, Diode_THT:D_DO-35_SOD27_P10.16mm_Horizontal
- removed Q3: BC337, Package_TO_SOT_THT:TO-92_Inline
- removed R10: 4k7, Resistor_THT:R_Axial_DIN0207_L6.3mm_D2.5mm_P10.16mm_Horizontal
- K1: value FINDER-32.21-x000 -> FINDER-40.52; footprint Relay_THT:Relay_SPDT_Finder_32.21-x000 -> Relay_THT:Relay_DPDT_Finder_40.52
- moved K1 8.00 mm to (164.4, 87.4)
- moved R5 6.36 mm to (179.7, 95.2)
- moved D3 6.36 mm to (176.5, 85.1)
- moved R11 6.35 mm to (173.4, 95.2)
- moved R6 6.35 mm to (183.5, 95.2)
- moved C1 5.08 mm to (176.5, 71.1)
- moved D1 5.08 mm to (154.9, 71.1)
- moved D2 5.08 mm to (173.4, 81.3)
- moved R1 5.08 mm to (151.1, 81.3)
- moved R2 5.08 mm to (179.7, 81.3)
- moved R3 5.08 mm to (170.2, 71.1)
- moved R9 5.08 mm to (183.5, 71.1)
- moved RV1 5.08 mm to (165.2, 81.3)
Connections:
- J4 pad 2: (no net) -> Net-(J4-Pad2)
- K1 pad 11: Net-(J1-Pad2) -> Net-(J4-Pad2)
- K1 pad 12: (no net) -> unconnected-(K1-Pad12)
- K1 pad 14: Net-(J1-Pad1) -> /Standby
Routing:
- net Net-(D3-Pad1): track 71.7 -> 44.4 mm
- net /Standby: track 28.5 -> 13.4 mm
- net Net-(Q3-Pad2): track 14.6 -> 0.00 mm
- net Net-(J4-Pad2): track 0.00 -> 9.13 mm
- net Net-(D2-Pad1): track 25.3 -> 21.6 mm
- net Net-(R11-Pad1): track 52.1 -> 48.6 mm
- net Net-(C2-Pad1): track 29.0 -> 25.8 mm
- net Net-(J1-Pad1): track 63.9 -> 66.7 mm
- net Net-(J1-Pad2): track 35.3 -> 37.0 mm
- net Net-(Q1-Pad3): track 5.23 -> 6.88 mm
- net Net-(Q2-Pad2): track 11.1 -> 10.5 mm
- net GND: vias 22 -> 14
Other:
- net class Default removed

Commit message: 6.3V, 400V und 400V Regler Boards bestellt
Parts:
- removed J6: Feedback, Connector_TE-Connectivity:TE_MATE-N-LOK_1-770866-x_1x02_P4.14mm_Vertical
- added SW1: Reset, Button_Switch_THT:SW_PUSH_6mm_H7.3mm, B.Cu at (138.5, 68.2)
- moved D5 7.01 mm to (144.1, 70.5)
Routing:
- net Net-(D2-K): track 21.6 -> 104.2 mm
- net Net-(D5-A): track 48.6 -> 45.1 mm
- net Net-(J1-Pin_1): track 66.7 -> 64.6 mm
- net +12V: track 11.5 -> 13.4 mm
- net Net-(Q2-C): track 25.8 -> 24.5 mm
- net Net-(Q1-E): track 6.88 -> 5.76 mm
- net GND: vias 14 -> 26
Other:
- board text removed: "Feedback"
