File: Boards/Bias/Bias.kicad_sch (KiCad schematic)
At the start: 34 parts

Commit message: 6.3V, 400V und 400V Regler Boards bestellt
Parts:
- added R2, R4: 10k, Resistor_THT:R_Axial_DIN0207_L6.3mm_D2.5mm_P10.16mm_Horizontal, symbol Device:R
- C1, C2, C3, C4, C5: value (none) -> 100nF; footprint (none) -> Capacitor_THT:C_Disc_D3.0mm_W2.0mm_P2.50mm
- D1: value (none) -> LED_ZV_R1; footprint (none) -> LED_THT:LED_D3.0mm
- D11, D15, D18, D23, D3, D6: value (none) -> 1N4148; footprint (none) -> Diode_THT:D_DO-35_SOD27_P10.16mm_Horizontal
- D13: value (none) -> LED_ZV_R2; footprint (none) -> LED_THT:LED_D3.0mm
- D17: value (none) -> LED_ZW_R2; footprint (none) -> LED_THT:LED_D3.0mm
- D19: value (none) -> LED_OK_R2; footprint (none) -> LED_THT:LED_D3.0mm
- D25: value (none) -> ZD5; footprint (none) -> Diode_THT:D_DO-41_SOD81_P10.16mm_Horizontal
- D5: value (none) -> LED_ZW_R1; footprint (none) -> LED_THT:LED_D3.0mm
- D7: value (none) -> LED_OK_R1; footprint (none) -> LED_THT:LED_D3.0mm
- J1: value (none) -> Conn_01x08; footprint (none) -> Connector_PinHeader_2.54mm:PinHeader_2x04_P2.54mm_Vertical
- R1, R11, R15, R19, R3, R7: value (none) -> 4k7; footprint (none) -> Resistor_THT:R_Axial_DIN0207_L6.3mm_D2.5mm_P10.16mm_Horizontal
- R17, R5: value (none) -> 1M; footprint (none) -> Resistor_THT:R_Axial_DIN0207_L6.3mm_D2.5mm_P10.16mm_Horizontal
- R21: value (none) -> 6k8; footprint (none) -> Resistor_THT:R_Axial_DIN0207_L6.3mm_D2.5mm_P10.16mm_Horizontal
- R22: value (none) -> 10k; footprint (none) -> Resistor_THT:R_Axial_DIN0207_L6.3mm_D2.5mm_P10.16mm_Horizontal
- R23: value (none) -> 60R4; footprint (none) -> Resistor_THT:R_Axial_DIN0207_L6.3mm_D2.5mm_P10.16mm_Horizontal
- R24: value (none) -> 562R; footprint (none) -> Resistor_THT:R_Axial_DIN0207_L6.3mm_D2.5mm_P10.16mm_Horizontal
- RV1, RV3: value (none) -> 10k; footprint (none) -> Potentiometer_THT:Potentiometer_Piher_PT-10-V10_Vertical_Hole
- U1: value (none) -> LM339; footprint (none) -> Package_DIP:DIP-14_W7.62mm
Connections:
- net GND: now also R2.2, R4.2; no longer RV1.1, RV3.1
- new net: R4.1, RV1.1
- new net: R2.1, RV3.1

Commit message: Leiterplatte erstellt
Parts:
- C1, C2, C3, C4, C5: footprint Capacitor_THT:C_Disc_D3.0mm_W2.0mm_P2.50mm -> Capacitor_THT:C_Disc_D4.3mm_W1.9mm_P5.00mm
- J1: footprint Connector_PinHeader_2.54mm:PinHeader_2x04_P2.54mm_Vertical -> Connector_IDC:IDC-Header_2x04_P2.54mm_Vertical
Changed lines of the file:
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@@
 			)
 		)
-		(property "Footprint" "Capacitor_THT:C_Disc_D3.0mm_W2.0mm_P2.50mm"
+		(property "Footprint" "Capacitor_THT:C_Disc_D4.3mm_W1.9mm_P5.00mm"
 			(at 120.65 63.5 0)
 			(effects
@@
 			)
 		)
-		(property "Footprint" "Capacitor_THT:C_Disc_D3.0mm_W2.0mm_P2.50mm"
+		(property "Footprint" "Capacitor_THT:C_Disc_D4.3mm_W1.9mm_P5.00mm"
 			(at 120.65 130.81 0)
 			(effects
@@
 			)
 		)
-		(property "Footprint" "Capacitor_THT:C_Disc_D3.0mm_W2.0mm_P2.50mm"
+		(property "Footprint" "Capacitor_THT:C_Disc_D4.3mm_W1.9mm_P5.00mm"
 			(at 38.1 36.83 0)
 			(effects
@@
 			)
 		)
-		(property "Footprint" "Capacitor_THT:C_Disc_D3.0mm_W2.0mm_P2.50mm"
+		(property "Footprint" "Capacitor_THT:C_Disc_D4.3mm_W1.9mm_P5.00mm"
 			(at 43.18 111.76 0)
 			(effects
@@
 			)
 		)
-		(property "Footprint" "Capacitor_THT:C_Disc_D3.0mm_W2.0mm_P2.50mm"
+		(property "Footprint" "Capacitor_THT:C_Disc_D4.3mm_W1.9mm_P5.00mm"
 			(at 43.18 93.98 0)
 			(effects
@@
 			)
 		)
-		(property "Footprint" "Connector_PinHeader_2.54mm:PinHeader_2x04_P2.54mm_Vertical"
+		(property "Footprint" "Connector_IDC:IDC-Header_2x04_P2.54mm_Vertical"
 			(at 69.85 97.79 0)
 			(effects
@@
 	)
 	(symbol
-		(lib_id "power:GND")
-		(at 81.28 110.49 0)
+		(lib_id "power:+12V")
+		(at 77.47 81.28 0)
 		(unit 1)
 		(exclude_from_sim no)
@@
 		(on_board yes)
 		(dnp no)
-		(property "Reference" "#PWR0101"
-			(at 81.28 116.84 0)
+		(property "Reference" "#PWR0102"
+			(at 77.47 85.09 0)
 			(effects
 				(font
@@
 			)
 		)
-		(property "Value" "GND"
-			(at 81.28 114.3 0)
+		(property "Value" "+12V"
+			(at 77.47 77.724 0)
 			(effects
 				(font
@@
 		)
 		(property "Footprint" ""
-			(at 81.28 110.49 0)
+			(at 77.47 81.28 0)
 			(effects
 				(font
@@
 		)
 		(property "Datasheet" ""
-			(at 81.28 110.49 0)
+			(at 77.47 81.28 0)
 			(effects
 				(font
@@
 		)
 		(property "Description" ""
-			(at 81.28 110.49 0)
+			(at 77.47 81.28 0)
 			(effects
 				(font
@@
 			(project "Bias"
 				(path "/842e430f-0c35-45f3-a0b5-95ae7b7ae388"
-					(reference "#PWR0101")
+					(reference "#PWR0102")
 					(unit 1)
 				)
@@
 	)
 	(symbol
-		(lib_id "power:+12V")
-		(at 77.47 81.28 0)
+		(lib_id "power:GND")
+		(at 88.9 99.06 0)
 		(unit 1)
 		(exclude_from_sim no)
@@
 		(on_board yes)
 		(dnp no)
-		(property "Reference" "#PWR0102"
-			(at 77.47 85.09 0)
+		(property "Reference" "#PWR0103"
+			(at 88.9 105.41 0)
 			(effects
 				(font
@@
 			)
 		)
-		(property "Value" "+12V"
-			(at 77.47 77.724 0)
+		(property "Value" "GND"
+			(at 88.9 102.87 0)
 			(effects
 				(font
@@
 		)
 		(property "Footprint" ""
-			(at 77.47 81.28 0)
+			(at 88.9 99.06 0)
 			(effects
 				(font
@@
 		)
 		(property "Datasheet" ""
-			(at 77.47 81.28 0)
+			(at 88.9 99.06 0)
 			(effects
 				(font
@@
 		)
 		(property "Description" ""
-			(at 77.47 81.28 0)
+			(at 88.9 99.06 0)
 			(effects
 				(font
@@
 			(project "Bias"
 				(path "/842e430f-0c35-45f3-a0b5-95ae7b7ae388"
-					(reference "#PWR0102")
+					(reference "#PWR0103")
 					(unit 1)
 				)
@@
 	(symbol
 		(lib_id "power:GND")
-		(at 88.9 99.06 0)
+		(at 101.6 120.65 0)
 		(unit 1)
 		(exclude_from_sim no)
@@
 		(on_board yes)
 		(dnp no)
-		(property "Reference" "#PWR0103"
-			(at 88.9 105.41 0)
+		(property "Reference" "#PWR08"
+			(at 101.6 127 0)
 			(effects
 				(font
@@
 		)
 		(property "Value" "GND"
-			(at 88.9 102.87 0)
+			(at 101.6 124.46 0)
 			(effects
 				(font
@@
 		)
 		(property "Footprint" ""
-			(at 88.9 99.06 0)
+			(at 101.6 120.65 0)
 			(effects
 				(font
@@
 		)
 		(property "Datasheet" ""
-			(at 88.9 99.06 0)
+			(at 101.6 120.65 0)
 			(effects
 				(font
@@
 		)
 		(property "Description" ""
-			(at 88.9 99.06 0)
+			(at 101.6 120.65 0)
 			(effects
 				(font
@@
 			(project "Bias"
 				(path "/842e430f-0c35-45f3-a0b5-95ae7b7ae388"
-					(reference "#PWR0103")
+					(reference "#PWR08")
 					(unit 1)
 				)
@@
 	(symbol
 		(lib_id "power:GND")
-		(at 101.6 87.63 0)
+		(at 81.28 110.49 0)
 		(unit 1)
 		(exclude_from_sim no)
@@
 		(on_board yes)
 		(dnp no)
-		(property "Reference" "#PWR0104"
-			(at 101.6 93.98 0)
+		(property "Reference" "#PWR07"
+			(at 81.28 116.84 0)
 			(effects
 				(font
@@
 		)
 		(property "Value" "GND"
-			(at 101.6 91.44 0)
+			(at 81.28 114.3 0)
 			(effects
 				(font
@@
 		)
 		(property "Footprint" ""
-			(at 101.6 87.63 0)
+			(at 81.28 110.49 0)
 			(effects
 				(font
@@
 		)
 		(property "Datasheet" ""
-			(at 101.6 87.63 0)
+			(at 81.28 110.49 0)
 			(effects
 				(font
@@
 		)
 		(property "Description" ""
-			(at 101.6 87.63 0)
+			(at 81.28 110.49 0)
 			(effects
 				(font
@@
 			(project "Bias"
 				(path "/842e430f-0c35-45f3-a0b5-95ae7b7ae388"
-					(reference "#PWR0104")
+					(reference "#PWR07")
 					(unit 1)
 				)
@@
 	(symbol
 		(lib_id "power:GND")
-		(at 101.6 120.65 0)
+		(at 101.6 87.63 0)
 		(unit 1)
 		(exclude_from_sim no)
@@
 		(on_board yes)
 		(dnp no)
-		(property "Reference" "#PWR0105"
-			(at 101.6 127 0)
+		(property "Reference" "#PWR09"
+			(at 101.6 93.98 0)
 			(effects
 				(font
@@
 		)
 		(property "Value" "GND"
-			(at 101.6 124.46 0)
+			(at 101.6 91.44 0)
 			(effects
 				(font
@@
 		)
 		(property "Footprint" ""
-			(at 101.6 120.65 0)
+			(at 101.6 87.63 0)
 			(effects
 				(font
@@
 		)
 		(property "Datasheet" ""
-			(at 101.6 120.65 0)
+			(at 101.6 87.63 0)
 			(effects
 				(font
@@
 		)
 		(property "Description" ""
-			(at 101.6 120.65 0)
+			(at 101.6 87.63 0)
 			(effects
 				(font
@@
 			(project "Bias"
 				(path "/842e430f-0c35-45f3-a0b5-95ae7b7ae388"
-					(reference "#PWR0105")
+					(reference "#PWR09")
 					(unit 1)
 				)
