File: Boards/Netzteil/12V_6V3_Delay/6V3.kicad_sch (KiCad schematic)
At the start: 40 parts, among them P6 7V5_AC, P7 6V3_DC_2, P8 6V3_DC_1, Q1 IRF530, Q2 IRF530, U2 LMC6482

Commit message: 6.3V, 400V und 400V Regler Boards bestellt
Parts:
- C15: footprint Capacitor_THT:CP_Radial_D35.0mm_P10.00mm_SnapIn -> Capacitor_THT:CP_Radial_D30.0mm_P10.00mm_SnapIn
- C22, C23, C9: footprint Capacitor_THT:C_Disc_D3.0mm_W2.0mm_P2.50mm -> Capacitor_THT:C_Disc_D4.3mm_W1.9mm_P5.00mm
- F2: footprint w_misc_comp:fuse_holder_CQ-2 -> Fuse_Holder_Eska:Fuse_Holder_Eska_509200
- P6, P7, P8: footprint Connector_TE-Connectivity:TE_MATE-N-LOK_1-770866-x_1x02_P4.14mm_Vertical -> Connector_Molex:Molex_Mini-Fit_Jr_5566-02A_2x01_P4.20mm_Vertical

Commit message: Leiterplatte erstellt
Parts:
- removed D13: LM385Z-1.2, Package_TO_SOT_THT:TO-92-2, symbol 6V3_Heizung-rescue:ZENER-RESCUE-6V3_Heizung
- added U5: LM385BZ-1.2, Package_TO_SOT_THT:TO-92_Inline, symbol Reference_Voltage:LM385BZ-1.2
- C10, C11, C12, C13: footprint Capacitor_THT:C_Disc_D3.0mm_W2.0mm_P2.50mm -> Capacitor_THT:C_Disc_D4.3mm_W1.9mm_P5.00mm
Connections:
- net GND: now also U5.3 (A)
- net Reference: now also U5.2 (K)
Changed lines of the file:
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@@
 	)
 	(junction
+		(at 139.7 88.9)
+		(diameter 0)
+		(color 0 0 0 0)
+	)
+	(junction
 		(at 238.76 99.06)
 		(diameter 0)
@@
 	)
 	(junction
-		(at 139.7 88.9)
-		(diameter 0)
-		(color 0 0 0 0)
-	)
-	(junction
 		(at 212.09 60.96)
 		(diameter 0)
@@
 	(wire
 		(pts
+			(xy 139.7 88.9) (xy 139.7 90.17)
+		)
+		(stroke
+			(width 0)
+			(type default)
+		)
+	)
+	(wire
+		(pts
 			(xy 222.25 99.06) (xy 229.87 99.06)
 		)
@@
 	(wire
 		(pts
+			(xy 139.7 97.79) (xy 139.7 99.06)
+		)
+		(stroke
+			(width 0)
+			(type default)
+		)
+	)
+	(wire
+		(pts
 			(xy 190.5 67.31) (xy 185.42 67.31)
 		)
@@
 	(wire
 		(pts
-			(xy 139.7 88.9) (xy 154.94 88.9)
-		)
-		(stroke
-			(width 0)
-			(type default)
-		)
-	)
-	(wire
-		(pts
 			(xy 161.29 93.98) (xy 161.29 105.41)
 		)
@@
 		)
 	)
+	(wire
+		(pts
+			(xy 139.7 88.9) (xy 154.94 88.9)
+		)
+		(stroke
+			(width 0)
+			(type default)
+		)
+	)
 	(text "9,21V"
 		(exclude_from_sim no)
@@
 			)
 		)
-		(property "Footprint" "Capacitor_THT:C_Disc_D3.0mm_W2.0mm_P2.50mm"
+		(property "Footprint" "Capacitor_THT:C_Disc_D4.3mm_W1.9mm_P5.00mm"
 			(at 77.1652 39.37 0)
 			(effects
@@
 			)
 		)
-		(property "Footprint" "Capacitor_THT:C_Disc_D3.0mm_W2.0mm_P2.50mm"
+		(property "Footprint" "Capacitor_THT:C_Disc_D4.3mm_W1.9mm_P5.00mm"
 			(at 77.1652 54.61 0)
 			(effects
@@
 			)
 		)
-		(property "Footprint" "Capacitor_THT:C_Disc_D3.0mm_W2.0mm_P2.50mm"
+		(property "Footprint" "Capacitor_THT:C_Disc_D4.3mm_W1.9mm_P5.00mm"
 			(at 102.5652 54.61 0)
 			(effects
@@
 			)
 		)
-		(property "Footprint" "Capacitor_THT:C_Disc_D3.0mm_W2.0mm_P2.50mm"
+		(property "Footprint" "Capacitor_THT:C_Disc_D4.3mm_W1.9mm_P5.00mm"
 			(at 102.5652 39.37 0)
 			(effects
@@
 	)
 	(symbol
-		(lib_id "6V3_Heizung-rescue:ZENER-RESCUE-6V3_Heizung")
-		(at 139.7 93.98 90)
-		(mirror x)
-		(unit 1)
-		(exclude_from_sim no)
-		(in_bom yes)
-		(on_board yes)
-		(dnp no)
-		(property "Reference" "D13"
-			(at 137.16 93.98 0)
-			(effects
-				(font
-					(size 1.27 1.27)
-				)
-			)
-		)
-		(property "Value" "LM385Z-1.2"
-			(at 142.24 93.98 90)
-			(effects
-				(font
-					(size 1.27 1.27)
-				)
-				(justify right)
-			)
-		)
-		(property "Footprint" "Package_TO_SOT_THT:TO-92-2"
-			(at 139.7 93.98 0)
-			(effects
-				(font
-					(size 1.524 1.524)
-				)
-				(hide yes)
-			)
-		)
-		(property "Datasheet" ""
-			(at 139.7 93.98 0)
-			(effects
-				(font
-					(size 1.524 1.524)
-				)
-			)
-		)
-		(property "Description" ""
-			(at 139.7 93.98 0)
-			(effects
-				(font
-					(size 1.27 1.27)
-				)
-				(hide yes)
-			)
-		)
-		(pin "1"
-		)
-		(pin "2"
-		)
-		(instances
-			(project "12V_6V3_Delay"
-				(path "/c034a787-71de-407a-b9e1-a8d5890447b1/00000000-0000-0000-0000-00006073a79d"
-					(reference "D13")
-					(unit 1)
-				)
-			)
-		)
-	)
-	(symbol
 		(lib_id "6V3_Heizung-rescue:GND-RESCUE-6V3_Heizung")
 		(at 127 101.6 0)
@@
 					(unit 1)
 				)
+			)
+		)
+	)
+	(symbol
+		(lib_id "Reference_Voltage:LM385BZ-1.2")
+		(at 139.7 93.98 90)
+		(unit 1)
+		(exclude_from_sim no)
+		(in_bom yes)
+		(on_board yes)
+		(dnp no)
+		(fields_autoplaced yes)
+		(property "Reference" "U5"
+			(at 141.7066 92.7678 90)
+			(effects
+				(font
+					(size 1.27 1.27)
+				)
+				(justify right)
+			)
+		)
+		(property "Value" "LM385BZ-1.2"
+			(at 141.7066 95.1921 90)
+			(effects
+				(font
+					(size 1.27 1.27)
+				)
+				(justify right)
+			)
+		)
+		(property "Footprint" "Package_TO_SOT_THT:TO-92_Inline"
+			(at 144.78 93.98 0)
+			(effects
+				(font
+					(size 1.27 1.27)
+					(italic yes)
+				)
+				(hide yes)
+			)
+		)
+		(property "Datasheet" "http://www.onsemi.com/pub_link/Collateral/LM285-D.PDF"
+			(at 139.7 93.98 0)
+			(effects
+				(font
+					(size 1.27 1.27)
+					(italic yes)
+				)
+				(hide yes)
+			)
+		)
+		(property "Description" "1.235V Micropower Voltage Reference Diodes, TO-92"
+			(at 139.7 93.98 0)
+			(effects
+				(font
+					(size 1.27 1.27)
+				)
+				(hide yes)
+			)
+		)
+		(pin "3"
+		)
+		(pin "2"
+		)
+		(instances
+			(project ""
+				(path "/c034a787-71de-407a-b9e1-a8d5890447b1/00000000-0000-0000-0000-00006073a79d"
+					(reference "U5")
+					(unit 1)
+				)
